File: Kicad Projects/7.0/BMS LTC6804-2/BMS LTC6804-2.kicad_pcb (KiCad board)
At the start: 2 copper layers, 85.1 x 85.1 mm, 74 parts, among them J1 CHG/DSCHG CTRL, J2 CHG/DSCHG CTRL CMP (SHORT DAT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, J3 Data IN/OUT, J4 Data IN/OUT, J5 Port Selector, J6 Port Selector, J7 NTC1, J8 NTC2, J9 Balance Connector, Q1 MMBT3906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

Commit message: Made both PCBs that should function for BMS Slave
Parts:
- added H1: MountingHole, MountingHole:MountingHole_3.2mm_M3, F.Cu at (104.2, 19.1)
- added H2: MountingHole, MountingHole:MountingHole_3.2mm_M3, B.Cu at (37.4, 19.1)
- added H3: MountingHole, MountingHole:MountingHole_3.2mm_M3, B.Cu at (37.6, 97.5)
- added H4: MountingHole, MountingHole:MountingHole_3.2mm_M3, F.Cu at (104.2, 97.5)
Routing:
- net DIN_GND: track 135.2 -> 141.9 mm
- net Net-(R2-Pad1): track 31.9 -> 35.8 mm
Changed lines of the file:
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@@
     )
   )
+  (footprint "MountingHole:MountingHole_3.2mm_M3" (layer "F.Cu")
+    (at 104.2162 19.1008)
+    (descr "Mounting Hole 3.2mm, no annular, M3")
+    (tags "mounting hole 3.2mm no annular m3")
+    (property "Sheetfile" "BMS LTC6804-2.kicad_sch")
+    (property "Sheetname" "")
+    (property "ki_description" "Mounting Hole without connection")
+    (property "ki_keywords" "mounting hole")
+    (attr exclude_from_pos_files)
+    (fp_text reference "H1" (at 0 -4.2) (layer "F.SilkS")
+        (effects (font (size 1 1) (thickness 0.15)))
+    )
+    (fp_text value "MountingHole" (at 0 4.2) (layer "F.Fab")
+        (effects (font (size 1 1) (thickness 0.15)))
+    )
+    (fp_text user "${REFERENCE}" (at 0 0) (layer "F.Fab")
+        (effects (font (size 1 1) (thickness 0.15)))
+    )
+    (fp_circle (center 0 0) (end 3.2 0)
+      (stroke (width 0.15) (type solid)) (fill none) (layer "Cmts.User"))
+    (fp_circle (center 0 0) (end 3.45 0)
+      (stroke (width 0.05) (type solid)) (fill none) (layer "F.CrtYd"))
+    (pad "" np_thru_hole circle (at 0 0) (size 3.2 3.2) (drill 3.2) (layers "F&B.Cu" "*.Mask")
+      (clearance 1.5))
+  )
   (footprint "Resistor_SMD:R_0805_2012Metric_Pad1.20x1.40mm_HandSolder" (layer "F.Cu")
     (at 39.8272 45.8724 90)
@@
     )
   )
+  (footprint "MountingHole:MountingHole_3.2mm_M3" (layer "F.Cu")
+    (at 104.2416 97.4852)
+    (descr "Mounting Hole 3.2mm, no annular, M3")
+    (tags "mounting hole 3.2mm no annular m3")
+    (property "Sheetfile" "BMS LTC6804-2.kicad_sch")
+    (property "Sheetname" "")
+    (property "ki_description" "Mounting Hole without connection")
+    (property "ki_keywords" "mounting hole")
+    (attr exclude_from_pos_files)
+    (fp_text reference "H4" (at 0 -4.2) (layer "F.SilkS")
+        (effects (font (size 1 1) (thickness 0.15)))
+    )
+    (fp_text value "MountingHole" (at 0 4.2) (layer "F.Fab")
+        (effects (font (size 1 1) (thickness 0.15)))
+    )
+    (fp_text user "${REFERENCE}" (at 0 0) (layer "F.Fab")
+        (effects (font (size 1 1) (thickness 0.15)))
+    )
+    (fp_circle (center 0 0) (end 3.2 0)
+      (stroke (width 0.15) (type solid)) (fill none) (layer "Cmts.User"))
+    (fp_circle (center 0 0) (end 3.45 0)
+      (stroke (width 0.05) (type solid)) (fill none) (layer "F.CrtYd"))
+    (pad "" np_thru_hole circle (at 0 0) (size 3.2 3.2) (drill 3.2) (layers "F&B.Cu" "*.Mask")
+      (clearance 1.5))
+  )
   (footprint "Package_SO:SOIC-4_4.55x3.7mm_P2.54mm" (layer "F.Cu")
     (at 45.391 53.2384)
@@
     )
   )
+  (footprint "MountingHole:MountingHole_3.2mm_M3" (layer "B.Cu")
+    (at 37.5666 97.4598 180)
+    (descr "Mounting Hole 3.2mm, no annular, M3")
+    (tags "mounting hole 3.2mm no annular m3")
+    (property "Sheetfile" "BMS LTC6804-2.kicad_sch")
+    (property "Sheetname" "")
+    (property "ki_description" "Mounting Hole without connection")
+    (property "ki_keywords" "mounting hole")
+    (attr exclude_from_pos_files)
+    (fp_text reference "H3" (at 0 4.2) (layer "B.SilkS")
+        (effects (font (size 1 1) (thickness 0.15)) (justify mirror))
+    )
+    (fp_text value "MountingHole" (at 0 -4.2) (layer "B.Fab")
+        (effects (font (size 1 1) (thickness 0.15)) (justify mirror))
+    )
+    (fp_text user "${REFERENCE}" (at 0 0) (layer "B.Fab")
+        (effects (font (size 1 1) (thickness 0.15)) (justify mirror))
+    )
+    (fp_circle (center 0 0) (end 3.2 0)
+      (stroke (width 0.15) (type solid)) (fill none) (layer "Cmts.User"))
+    (fp_circle (center 0 0) (end 3.45 0)
+      (stroke (width 0.05) (type solid)) (fill none) (layer "B.CrtYd"))
+    (pad "" np_thru_hole circle (at 0 0 180) (size 3.2 3.2) (drill 3.2) (layers "F&B.Cu" "*.Mask")
+      (clearance 1.5))
+  )
   (footprint "Capacitor_SMD:C_0805_2012Metric_Pad1.18x1.45mm_HandSolder" (layer "B.Cu")
     (at 85.852 62.103 -90)
@@
     )
   )
+  (footprint "MountingHole:MountingHole_3.2mm_M3" (layer "B.Cu")
+    (at 37.3634 19.1008 180)
+    (descr "Mounting Hole 3.2mm, no annular, M3")
+    (tags "mounting hole 3.2mm no annular m3")
+    (property "Sheetfile" "BMS LTC6804-2.kicad_sch")
+    (property "Sheetname" "")
+    (property "ki_description" "Mounting Hole without connection")
+    (property "ki_keywords" "mounting hole")
+    (attr exclude_from_pos_files)
+    (fp_text reference "H2" (at 0 4.2) (layer "B.SilkS")
+        (effects (font (size 1 1) (thickness 0.15)) (justify mirror))
+    )
+    (fp_text value "MountingHole" (at 0 -4.2) (layer "B.Fab")
+        (effects (font (size 1 1) (thickness 0.15)) (justify mirror))
+    )
+    (fp_text user "${REFERENCE}" (at 0 0) (layer "B.Fab")
+        (effects (font (size 1 1) (thickness 0.15)) (justify mirror))
+    )
+    (fp_circle (center 0 0) (end 3.2 0)
+      (stroke (width 0.15) (type solid)) (fill none) (layer "Cmts.User"))
+    (fp_circle (center 0 0) (end 3.45 0)
+      (stroke (width 0.05) (type solid)) (fill none) (layer "B.CrtYd"))
+    (pad "" np_thru_hole circle (at 0 0 180) (size 3.2 3.2) (drill 3.2) (layers "F&B.Cu" "*.Mask")
+      (clearance 1.5))
+  )
   (footprint "Capacitor_SMD:C_0805_2012Metric_Pad1.18x1.45mm_HandSolder" (layer "B.Cu")
     (at 85.725 66.421 -90)
@@
   (via (at 41.3766 43.7642) (size 0.8) (drill 0.4) (layers "F.Cu" "B.Cu") (net 34))
   (via (at 29.3395 89.6874) (size 0.8) (drill 0.4) (layers "F.Cu" "B.Cu") (net 34))
+  (segment (start 26.329 92.384) (end 26.329 98.2872) (width 0.25) (layer "B.Cu") (net 34))
+  (segment (start 26.8732 98.8314) (end 31.1912 98.8314) (width 0.25) (layer "B.Cu") (net 34))
   (segment (start 41.9393 44.3269) (end 41.3766 43.7642) (width 0.25) (layer "B.Cu") (net 34))
-  (segment (start 26.329 98.2872) (end 26.8732 98.8314) (width 0.25) (layer "B.Cu") (net 34))
   (segment (start 29.3395 89.6874) (end 28.6258 89.6874) (width 0.25) (layer "B.Cu") (net 34))
-  (segment (start 26.8732 98.8314) (end 61.8744 98.8314) (width 0.25) (layer "B.Cu") (net 34))
+  (segment (start 43.6626 96.5454) (end 43.6626 96.6216) (width 0.25) (layer "B.Cu") (net 34))
+  (segment (start 39.9288 92.8116) (end 43.6626 96.5454) (width 0.25) (layer "B.Cu") (net 34))
+  (segment (start 32.5556 94.4952) (end 34.2392 92.8116) (width 0.25) (layer "B.Cu") (net 34))
+  (segment (start 32.5556 97.467) (end 32.5556 94.4952) (width 0.25) (layer "B.Cu") (net 34))
   (segment (start 41.3766 43.7642) (end 29.4919 43.7642) (width 0.25) (layer "B.Cu") (net 34))
+  (segment (start 45.8724 98.8314) (end 61.8744 98.8314) (width 0.25) (layer "B.Cu") (net 34))
   (segment (start 43.7642 44.3269) (end 41.9393 44.3269) (width 0.25) (layer "B.Cu") (net 34))
   (segment (start 29.4919 43.7642) (end 29.3395 43.9166) (width 0.25) (layer "B.Cu") (net 34))
+  (segment (start 31.1912 98.8314) (end 32.5556 97.467) (width 0.25) (layer "B.Cu") (net 34))
+  (segment (start 34.2392 92.8116) (end 39.9288 92.8116) (width 0.25) (layer "B.Cu") (net 34))
+  (segment (start 43.6626 96.6216) (end 45.8724 98.8314) (width 0.25) (layer "B.Cu") (net 34))
   (segment (start 28.6258 89.6874) (end 27.3812 90.932) (width 0.25) (layer "B.Cu") (net 34))
-  (segment (start 26.329 92.384) (end 26.329 98.2872) (width 0.25) (layer "B.Cu") (net 34))
+  (segment (start 26.329 98.2872) (end 26.8732 98.8314) (width 0.25) (layer "B.Cu") (net 34))
   (segment (start 79.8322 50.9016) (end 79.8322 52.114812) (width 0.25) (layer "F.Cu") (net 35))
   (segment (start 79.973 91.1191) (end 79.973 52.5642) (width 0.25) (layer "F.Cu") (net 35))
@@
   (segment (start 37.3126 52.1462) (end 41.9632 52.1462) (width 0.25) (layer "B.Cu") (net 65))
   (via (at 62.5868 96.2914) (size 0.8) (drill 0.4) (layers "F.Cu" "B.Cu") (net 66))
+  (segment (start 32.1056 95.4786) (end 32.1056 94.1324) (width 0.25) (layer "B.Cu") (net 66))
   (segment (start 62.3074 96.012) (end 62.5868 96.2914) (width 0.25) (layer "B.Cu") (net 66))
-  (segment (start 30.845 96.012) (end 62.3074 96.012) (width 0.25) (layer "B.Cu") (net 66))
+  (segment (start 40.2844 92.2274) (end 44.069 96.012) (width 0.25) (layer "B.Cu") (net 66))
+  (segment (start 32.1056 94.1324) (end 34.0106 92.2274) (width 0.25) (layer "B.Cu") (net 66))
+  (segment (start 30.845 96.012) (end 31.5722 96.012) (width 0.25) (layer "B.Cu") (net 66))
+  (segment (start 44.069 96.012) (end 62.3074 96.012) (width 0.25) (layer "B.Cu") (net 66))
+  (segment (start 34.0106 92.2274) (end 40.2844 92.2274) (width 0.25) (layer "B.Cu") (net 66))
+  (segment (start 31.5722 96.012) (end 32.1056 95.4786) (width 0.25) (layer "B.Cu") (net 66))
   (segment (start 40.4368 39.1668) (end 42.7116 39.1668) (width 0.25) (layer "F.Cu") (net 67))
   (segment (start 71.4916 91.2368) (end 71.5932 91.3384) (width 0.25) (layer "F.Cu") (net 68))

Commit message: IDEK
Routing:
- net Net-(U9-S6): track 14.0 -> 13.3 mm
Changed lines of the file:
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@@
   (segment (start 84.802 57.082764) (end 84.802 55.0219) (width 0.25) (layer "B.Cu") (net 38))
   (segment (start 83.694764 58.19) (end 84.802 57.082764) (width 0.25) (layer "B.Cu") (net 38))
-  (segment (start 87.1474 56.515) (end 87.6808 56.515) (width 0.25) (layer "F.Cu") (net 39))
-  (segment (start 87.884 56.3118) (end 87.884 54.8855) (width 0.25) (layer "F.Cu") (net 39))
-  (segment (start 85.965989 57.023) (end 86.6394 57.023) (width 0.25) (layer "F.Cu") (net 39))
-  (segment (start 86.6394 57.023) (end 87.1474 56.515) (width 0.25) (layer "F.Cu") (net 39))
-  (segment (start 87.6808 56.515) (end 87.884 56.3118) (width 0.25) (layer "F.Cu") (net 39))
-  (segment (start 84.592032 58.396957) (end 85.965989 57.023) (width 0.25) (layer "F.Cu") (net 39))
+  (segment (start 86.473989 56.515) (end 84.592032 58.396957) (width 0.25) (layer "F.Cu") (net 39))
+  (segment (start 87.884 56.3118) (end 87.6808 56.515) (width 0.25) (layer "F.Cu") (net 39))
+  (segment (start 87.6808 56.515) (end 86.473989 56.515) (width 0.25) (layer "F.Cu") (net 39))
+  (segment (start 87.884 54.8855) (end 87.884 56.3118) (width 0.25) (layer "F.Cu") (net 39))
   (via (at 84.592032 58.396957) (size 0.8) (drill 0.4) (layers "F.Cu" "B.Cu") (net 39))
   (via (at 87.503 54.864) (size 0.8) (drill 0.4) (layers "F.Cu" "B.Cu") (net 39))
@@
   (segment (start 85.076061 58.936047) (end 85.098047 58.936047) (width 0.25) (layer "B.Cu") (net 77))
   (segment (start 82.677 59.69) (end 84.322108 59.69) (width 0.25) (layer "B.Cu") (net 77))
-  (segment (start 85.461695 56.3372) (end 86.614 56.3372) (width 0.25) (layer "F.Cu") (net 78))
   (segment (start 86.614 54.5229) (end 87.1639 53.973) (width 0.25) (layer "F.Cu") (net 78))
+  (segment (start 86.614 55.245) (end 85.5218 56.3372) (width 0.25) (layer "F.Cu") (net 78))
+  (segment (start 85.5218 56.3372) (end 85.461695 56.3372) (width 0.25) (layer "F.Cu") (net 78))
   (segment (start 89.041 53.973) (end 89.932 54.864) (width 0.25) (layer "F.Cu") (net 78))
   (segment (start 82.814216 58.984679) (end 85.461695 56.3372) (width 0.25) (layer "F.Cu") (net 78))
   (segment (start 87.1639 53.973) (end 89.041 53.973) (width 0.25) (layer "F.Cu") (net 78))
+  (segment (start 86.614 55.245) (end 86.614 54.5229) (width 0.25) (layer "F.Cu") (net 78))
   (segment (start 81.140208 58.984679) (end 82.814216 58.984679) (width 0.25) (layer "F.Cu") (net 78))
-  (segment (start 86.614 56.3372) (end 86.614 54.5229) (width 0.25) (layer "F.Cu") (net 78))
   (via (at 81.140208 58.984679) (size 0.8) (drill 0.4) (layers "F.Cu" "B.Cu") (net 78))
   (segment (start 81.434887 58.69) (end 82.677 58.69) (width 0.25) (layer "B.Cu") (net 78))
   (segment (start 81.140208 58.984679) (end 81.434887 58.69) (width 0.25) (layer "B.Cu") (net 78))
-  (segment (start 86.106 55.8546) (end 86.106 54.394504) (width 0.25) (layer "F.Cu") (net 79))
-  (segment (start 85.307899 55.8546) (end 86.106 55.8546) (width 0.25) (layer "F.Cu") (net 79))
-  (segment (start 86.106 54.394504) (end 86.912652 53.587852) (width 0.25) (layer "F.Cu") (net 79))
-  (segment (start 81.137603 57.498014) (end 83.664485 57.498014) (width 0.25) (layer "F.Cu") (net 79))
-  (segment (start 86.834 53.5092) (end 86.834 51.739) (width 0.25) (layer "F.Cu") (net 79))
-  (segment (start 86.912652 53.587852) (end 86.834 53.5092) (width 0.25) (layer "F.Cu") (net 79))
-  (segment (start 83.664485 57.498014) (end 85.307899 55.8546) (width 0.25) (layer "F.Cu") (net 79))
-  (segment (start 86.834 51.739) (end 87.9 50.673) (width 0.25) (layer "F.Cu") (net 79))
+  (segment (start 86.834 51.739) (end 86.834 53.5092) (width 0.25) (layer "F.Cu") (net 79))
+  (segment (start 85.3694 55.8546) (end 85.307899 55.8546) (width 0.25) (layer "F.Cu") (net 79))
+  (segment (start 86.834 53.5092) (end 86.912652 53.587852) (width 0.25) (layer "F.Cu") (net 79))
+  (segment (start 83.664485 57.498014) (end 81.137603 57.498014) (width 0.25) (layer "F.Cu") (net 79))
+  (segment (start 87.9 50.673) (end 86.834 51.739) (width 0.25) (layer "F.Cu") (net 79))
+  (segment (start 86.912652 53.587852) (end 86.106 54.394504) (width 0.25) (layer "F.Cu") (net 79))
+  (segment (start 86.106 54.394504) (end 86.106 55.118) (width 0.25) (layer "F.Cu") (net 79))
+  (segment (start 86.106 55.118) (end 85.3694 55.8546) (width 0.25) (layer "F.Cu") (net 79))
+  (segment (start 85.307899 55.8546) (end 83.664485 57.498014) (width 0.25) (layer "F.Cu") (net 79))
   (via (at 81.137603 57.498014) (size 0.8) (drill 0.4) (layers "F.Cu" "B.Cu") (net 79))
   (segment (start 81.445617 57.19) (end 81.137603 57.498014) (width 0.25) (layer "B.Cu") (net 79))
   (segment (start 82.677 57.19) (end 81.445617 57.19) (width 0.25) (layer "B.Cu") (net 79))
   (segment (start 82.677 57.19) (end 83.694764 57.19) (width 0.25) (layer "B.Cu") (net 79))
+  (segment (start 85.8012 48.6664) (end 85.5218 48.9458) (width 0.25) (layer "F.Cu") (net 80))
+  (segment (start 86.106 53.4924) (end 85.4202 54.1782) (width 0.25) (layer "F.Cu") (net 80))
+  (segment (start 85.8012 47.3335) (end 85.8012 48.6664) (width 0.25) (layer "F.Cu") (net 80))
   (segment (start 86.106 50.8254) (end 86.106 53.4924) (width 0.25) (layer "F.Cu") (net 80))
-  (segment (start 84.201 56.134) (end 84.0232 56.3118) (width 0.25) (layer "F.Cu") (net 80))
-  (segment (start 86.106 53.4924) (end 85.8266 53.7718) (width 0.25) (layer "F.Cu") (net 80))
-  (segment (start 85.8012 48.6664) (end 85.5218 48.9458) (width 0.25) (layer "F.Cu") (net 80))
-  (segment (start 85.8012 47.3335) (end 85.8012 48.6664) (width 0.25) (layer "F.Cu") (net 80))
-  (segment (start 84.9884 55.3466) (end 84.201 56.134) (width 0.25) (layer "F.Cu") (net 80))
-  (segment (start 85.8266 53.7718) (end 85.4202 54.1782) (width 0.25) (layer "F.Cu") (net 80))
-  (segment (start 85.4202 55.3466) (end 84.9884 55.3466) (width 0.25) (layer "F.Cu") (net 80))
+  (segment (start 85.4202 54.1782) (end 85.4202 54.9148) (width 0.25) (layer "F.Cu") (net 80))
   (segment (start 84.0232 56.3118) (end 81.1784 56.3118) (width 0.25) (layer "F.Cu") (net 80))
-  (segment (start 85.4202 54.1782) (end 85.4202 55.3466) (width 0.25) (layer "F.Cu") (net 80))
+  (segment (start 85.4202 54.9148) (end 84.0232 56.3118) (width 0.25) (layer "F.Cu") (net 80))
   (via (at 86.106 50.8254) (size 0.8) (drill 0.4) (layers "F.Cu" "B.Cu") (net 80))
   (via (at 85.5218 48.9458) (size 0.8) (drill 0.4) (layers "F.Cu" "B.Cu") (net 80))
@@
   (segment (start 86.4268 52.1462) (end 87.9 50.673) (width 0.25) (layer "B.Cu") (net 81))
   (segment (start 85.5472 52.1462) (end 86.4268 52.1462) (width 0.25) (layer "B.Cu") (net 81))
+  (segment (start 85.159 50.7674) (end 85.159 50.5786) (width 0.25) (layer "F.Cu") (net 82))
+  (segment (start 85.1662 52.071396) (end 85.1662 50.7746) (width 0.25) (layer "F.Cu") (net 82))
+  (segment (start 87.0966 48.641) (end 87.9 48.641) (width 0.25) (layer "F.Cu") (net 82))
+  (segment (start 84.126196 53.1114) (end 85.1662 52.071396) (width 0.25) (layer "F.Cu") (net 82))
+  (segment (start 85.159 50.5786) (end 87.0966 48.641) (width 0.25) (layer "F.Cu") (net 82))
+  (segment (start 82.061777 53.1114) (end 84.126196 53.1114) (width 0.25) (layer "F.Cu") (net 82))
+  (segment (start 85.1662 50.7746) (end 85.159 50.7674) (width 0.25) (layer "F.Cu") (net 82))
   (segment (start 81.169585 54.003592) (end 82.061777 53.1114) (width 0.25) (layer "F.Cu") (net 82))
-  (segment (start 85.1662 52.071396) (end 85.1662 50.7746) (width 0.25) (layer "F.Cu") (net 82))
-  (segment (start 85.1662 50.7746) (end 85.159 50.7674) (width 0.25) (layer "F.Cu") (net 82))
-  (segment (start 85.159 49.8094) (end 85.9282 49.8094) (width 0.25) (layer "F.Cu") (net 82))
-  (segment (start 82.061777 53.1114) (end 84.126196 53.1114) (width 0.25) (layer "F.Cu") (net 82))
-  (segment (start 85.9282 49.8094) (end 87.0966 48.641) (width 0.25) (layer "F.Cu") (net 82))
-  (segment (start 84.126196 53.1114) (end 85.1662 52.071396) (width 0.25) (layer "F.Cu") (net 82))
-  (segment (start 87.0966 48.641) (end 87.9 48.641) (width 0.25) (layer "F.Cu") (net 82))
-  (segment (start 85.159 50.7674) (end 85.159 49.8094) (width 0.25) (layer "F.Cu") (net 82))
   (via (at 81.169585 54.003592) (size 0.8) (drill 0.4) (layers "F.Cu" "B.Cu") (net 82))
   (segment (start 81.169585 54.003592) (end 81.355993 54.19) (width 0.25) (layer "B.Cu") (net 82))
