File: Kicad Projects/7.0/Levitation Unit/LU/LU.kicad_pcb (KiCad board)
At the start: 2 copper layers, 95 parts, among them IC1 1ED3322MC12NXUMA1, IC2 B0505S-2W, IC3 B0505S-2W, IC4 B0505S-2W, IC5 1ED3322MC12NXUMA1, J1 Conn_01x02_Male, J2 Conn_01x04_Pin, J3 Conn_01x02_Male, U1 LM7809_TO220, U10 6N137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

Commit message: Inverter 0 errors ready to export, LU fucked
Parts:
- added Q1: F4-75R06W1E3, IGBT:F475R06W1E3, F.Cu at (191.6, 61.0)
- U7: moved to B.Cu
- turned U7 to 180 degrees
Connections:
- R1 pad 2: Net-(R1-Pad2) -> unconnected-(R1-Pad2)
- R3 pad 2: Net-(R3-Pad2) -> unconnected-(R3-Pad2)
Routing:
- net Net-(Q1-PadEU1): track 0.00 -> 92.0 mm
- net Net-(Q1-PadU1): track 0.00 -> 89.6 mm
- net Net-(Q1-PadE2): track 0.00 -> 27.3 mm
- net Net-(Q1-PadG2): track 0.00 -> 27.2 mm
- net Net-(Q1-PadG1): track 0.00 -> 25.6 mm
- net Net-(Q1-PadE1): track 0.00 -> 25.6 mm
- net Net-(Q1-PadP1): track 0.00 -> 6.40 mm
- net Net-(Q1-PadT1): track 0.00 -> 6.40 mm
