File: Kicad Projects/7.0/Chg_Dschg Controller/Chg_Dschg Controller.kicad_pcb (KiCad board)
At the start: 2 copper layers, 99 parts, among them J1 Slave socket, J10 Boost OUT, J2 Electronics, J3 Charger, J4 Battery, J5 Contactor, J6 NO/NC Contactor, J7 NC/NO Charge, J8 NO/NC Charge-, J9 NO/NC Charge+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

Commit message: Inverter gbr generated
Connections:
- net Net-(J6-Pin_1) renamed /NOR1
- net Net-(J6-Pin_3) renamed /NCR1
Changed lines of the file:
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@@
   (net 13 "Net-(J4-Pin_1)")
   (net 14 "-BATT")
-  (net 15 "Net-(J6-Pin_1)")
-  (net 16 "Net-(J6-Pin_3)")
+  (net 15 "/NOR1")
+  (net 16 "/NCR1")
   (net 17 "Net-(J7-Pin_2)")
   (net 18 "Net-(J8-Pin_1)")
@@
       (stroke (width 0.1) (type solid)) (layer "F.Fab"))
     (pad "1" thru_hole rect (at 0 0) (size 0.85 0.85) (drill 0.5) (layers "*.Cu" "*.Mask")
-      (net 15 "Net-(J6-Pin_1)") (pinfunction "Pin_1") (pintype "passive"))
+      (net 15 "/NOR1") (pinfunction "Pin_1") (pintype "passive"))
     (pad "2" thru_hole oval (at 0 1) (size 0.85 0.85) (drill 0.5) (layers "*.Cu" "*.Mask")
       (net 2 "Net-(D1-A)") (pinfunction "Pin_2") (pintype "passive"))
     (pad "3" thru_hole oval (at 0 2) (size 0.85 0.85) (drill 0.5) (layers "*.Cu" "*.Mask")
-      (net 16 "Net-(J6-Pin_3)") (pinfunction "Pin_3") (pintype "passive"))
+      (net 16 "/NCR1") (pinfunction "Pin_3") (pintype "passive"))
     (model "${KICAD6_3DMODEL_DIR}/Connector_PinHeader_1.00mm.3dshapes/PinHeader_1x03_P1.00mm_Vertical.wrl"
       (offset (xyz 0 0 0))
@@
       (net 4 "Net-(D3-A)") (pintype "passive"))
     (pad "3" thru_hole oval (at -6 14.2) (size 2.5 2.5) (drill 1.3) (layers "*.Cu" "*.Mask")
-      (net 16 "Net-(J6-Pin_3)") (pintype "passive"))
+      (net 16 "/NCR1") (pintype "passive"))
     (pad "4" thru_hole oval (at 6 14.2) (size 2.5 2.5) (drill 1.3) (layers "*.Cu" "*.Mask")
-      (net 15 "Net-(J6-Pin_1)") (pintype "passive"))
+      (net 15 "/NOR1") (pintype "passive"))
     (pad "5" thru_hole oval (at 6 2) (size 2.5 2.5) (drill 1.3) (layers "*.Cu" "*.Mask")
       (net 29 "/12V") (pintype "passive"))
@@
       (stroke (width 0.1) (type solid)) (layer "F.Fab"))
     (pad "1" thru_hole rect (at 0 0) (size 0.85 0.85) (drill 0.5) (layers "*.Cu" "*.Mask")
-      (net 15 "Net-(J6-Pin_1)") (pinfunction "Pin_1") (pintype "passive"))
+      (net 15 "/NOR1") (pinfunction "Pin_1") (pintype "passive"))
     (pad "2" thru_hole oval (at 0 1) (size 0.85 0.85) (drill 0.5) (layers "*.Cu" "*.Mask")
       (net 17 "Net-(J7-Pin_2)") (pinfunction "Pin_2") (pintype "passive"))
     (pad "3" thru_hole oval (at 0 2) (size 0.85 0.85) (drill 0.5) (layers "*.Cu" "*.Mask")
-      (net 16 "Net-(J6-Pin_3)") (pinfunction "Pin_3") (pintype "passive"))
+      (net 16 "/NCR1") (pinfunction "Pin_3") (pintype "passive"))
     (model "${KICAD6_3DMODEL_DIR}/Connector_PinHeader_1.00mm.3dshapes/PinHeader_1x03_P1.00mm_Vertical.wrl"
       (offset (xyz 0 0 0))
