File: Kicad Projects/7.0/Chg_Dschg Controller/Chg_Dschg Controller.kicad_sch (KiCad schematic)
At the start: 99 parts, among them J1 Slave socket, J10 Boost OUT, J2 Electronics, J3 Charger, J4 Battery, J5 Contactor, J6 NO/NC Contactor, J7 NC/NO Charge, J8 NO/NC Charge-, J9 NO/NC Charge+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

Commit message: Inverter gbr generated
Parts:
- added D10, D11: D_Zener, Diode_SMD:D_SMA_Handsoldering, symbol Device:D_Zener
- R56: value 1k -> 10k
Connections:
- net -BATT: now also D11.2 (A)
- net Gate1: now also D11.1 (K)
- net NOR1: now reaches J6.3 (Pin_3), J7.3 (Pin_3), K1.3
- net NCR1: now reaches J6.1 (Pin_1), J7.1 (Pin_1), K1.4
- net at D14.2 (A), J1.5 (Pin_5), Q1.1 (G)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: now also D10.1 (K), D10.2 (A)
Changed lines of the file:
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@@
   (junction (at 118.11 130.81) (diameter 0) (color 0 0 0 0)
   )
+  (junction (at 92.71 40.64) (diameter 0) (color 0 0 0 0)
+  )
   (junction (at 130.81 130.81) (diameter 0) (color 0 0 0 0)
   )
@@
   (junction (at 86.36 36.83) (diameter 0) (color 0 0 0 0)
   )
+  (junction (at 82.55 36.83) (diameter 0) (color 0 0 0 0)
+  )
   (junction (at 77.47 144.78) (diameter 0) (color 0 0 0 0)
   )
@@
   (junction (at 130.81 143.51) (diameter 0) (color 0 0 0 0)
   )
+  (junction (at 91.44 59.69) (diameter 0) (color 0 0 0 0)
+  )
   (junction (at 125.73 104.14) (diameter 0) (color 0 0 0 0)
   )
@@
     (stroke (width 0) (type default))
   )
+  (wire (pts (xy 91.44 67.31) (xy 101.6 67.31))
+    (stroke (width 0) (type default))
+  )
   (wire (pts (xy 171.45 62.23) (xy 167.64 62.23))
     (stroke (width 0) (type default))
@@
     (stroke (width 0) (type default))
   )
+  (wire (pts (xy 82.55 36.83) (xy 86.36 36.83))
+    (stroke (width 0) (type default))
+  )
   (wire (pts (xy 114.3 143.51) (xy 125.73 143.51))
     (stroke (width 0) (type default))
@@
     (stroke (width 0) (type default))
   )
+  (wire (pts (xy 82.55 44.45) (xy 92.71 44.45))
+    (stroke (width 0) (type default))
+  )
   (wire (pts (xy 113.03 139.7) (xy 114.3 139.7))
     (stroke (width 0) (type default))
@@
     (stroke (width 0) (type default))
   )
+  (wire (pts (xy 92.71 40.64) (xy 142.24 40.64))
+    (stroke (width 0) (type default))
+  )
   (wire (pts (xy 123.19 99.06) (xy 124.46 99.06))
     (stroke (width 0) (type default))
@@
     (stroke (width 0) (type default))
   )
+  (wire (pts (xy 92.71 40.64) (xy 92.71 44.45))
+    (stroke (width 0) (type default))
+  )
   (wire (pts (xy 77.47 149.86) (xy 77.47 156.21))
     (stroke (width 0) (type default))
@@
     (stroke (width 0) (type default))
   )
+  (wire (pts (xy 99.06 59.69) (xy 101.6 59.69))
+    (stroke (width 0) (type default))
+  )
   (wire (pts (xy 34.29 60.96) (xy 90.17 60.96))
     (stroke (width 0) (type default))
@@
     (stroke (width 0) (type default))
   )
-  (wire (pts (xy 86.36 40.64) (xy 142.24 40.64))
+  (wire (pts (xy 86.36 40.64) (xy 92.71 40.64))
     (stroke (width 0) (type default))
   )
@@
     (stroke (width 0) (type default))
   )
+  (wire (pts (xy 101.6 59.69) (xy 101.6 67.31))
+    (stroke (width 0) (type default))
+  )
   (wire (pts (xy 187.96 66.04) (xy 187.96 62.23))
     (stroke (width 0) (type default))
@@
     (stroke (width 0) (type default))
   )
-  (wire (pts (xy 68.58 36.83) (xy 86.36 36.83))
+  (wire (pts (xy 68.58 36.83) (xy 82.55 36.83))
     (stroke (width 0) (type default))
   )
@@
     (stroke (width 0) (type default))
   )
+  (label "NOR1" (at 201.93 13.97 0) (fields_autoplaced)
+    (effects (font (size 1.27 1.27)) (justify left bottom))
+  )
   (label "Drain1" (at 99.06 48.26 0) (fields_autoplaced)
     (effects (font (size 1.27 1.27)) (justify left bottom))
   )
+  (label "NCR1" (at 207.01 15.24 0) (fields_autoplaced)
+    (effects (font (size 1.27 1.27)) (justify left bottom))
+  )
   (label "5V" (at 36.83 63.5 0) (fields_autoplaced)
     (effects (font (size 1.27 1.27)) (justify left bottom))
@@
     )
   )
+  (symbol (lib_id "Device:D_Zener") (at 82.55 40.64 270) (unit 1)
+    (in_bom yes) (on_board yes) (dnp no) (fields_autoplaced)
+    (property "Reference" "D10" (at 85.09 39.37 90)
+      (effects (font (size 1.27 1.27)) (justify left))
+    )
+    (property "Value" "D_Zener" (at 85.09 41.91 90)
+      (effects (font (size 1.27 1.27)) (justify left))
+    )
+    (property "Footprint" "Diode_SMD:D_SMA_Handsoldering" (at 82.55 40.64 0)
+      (effects (font (size 1.27 1.27)) hide)
+    )
+    (property "Datasheet" "~" (at 82.55 40.64 0)
+      (effects (font (size 1.27 1.27)) hide)
+    )
+    (pin "1")
+    (pin "2")
+    (instances
+      (project "Chg_Dschg Controller"
+        (path "/44b4c7bd-7876-4094-a297-c391da939751"
+          (reference "D10") (unit 1)
+        )
+      )
+    )
+  )
   (symbol (lib_id "Device:R") (at 144.78 191.77 90) (unit 1)
     (in_bom yes) (on_board yes) (dnp no) (fields_autoplaced)
@@
     )
   )
+  (symbol (lib_id "Device:D_Zener") (at 91.44 63.5 270) (unit 1)
+    (in_bom yes) (on_board yes) (dnp no) (fields_autoplaced)
+    (property "Reference" "D11" (at 93.98 62.23 90)
+      (effects (font (size 1.27 1.27)) (justify left))
+    )
+    (property "Value" "D_Zener" (at 93.98 64.77 90)
+      (effects (font (size 1.27 1.27)) (justify left))
+    )
+    (property "Footprint" "Diode_SMD:D_SMA_Handsoldering" (at 91.44 63.5 0)
+      (effects (font (size 1.27 1.27)) hide)
+    )
+    (property "Datasheet" "~" (at 91.44 63.5 0)
+      (effects (font (size 1.27 1.27)) hide)
+    )
+    (pin "1")
+    (pin "2")
+    (instances
+      (project "Chg_Dschg Controller"
+        (path "/44b4c7bd-7876-4094-a297-c391da939751"
+          (reference "D11") (unit 1)
+        )
+      )
+    )
+  )
   (symbol (lib_id "Device:R") (at 121.92 171.45 0) (unit 1)
     (in_bom yes) (on_board yes) (dnp no) (fields_autoplaced)
@@
       (effects (font (size 1.27 1.27)) (justify left))
     )
-    (property "Value" "1k" (at 74.93 54.61 0)
+    (property "Value" "10k" (at 74.93 54.61 0)
       (effects (font (size 1.27 1.27)) (justify left))
     )
@@
       (effects (font (size 1.27 1.27)) (justify left))
     )
-    (property "Value" "1k" (at 71.12 33.02 0)
+    (property "Value" "10k" (at 71.12 33.02 0)
       (effects (font (size 1.27 1.27)) (justify left))
     )
