File: Vegapod 24/Kicad Projects/7.0/Inverter/Inverter/Inverter.kicad_pcb (KiCad board)
At the start: 4 copper layers, 80.3 x 134.5 mm, 122 parts, among them IC1 1ED3322MC12NXUMA1, IC2 B0505S-2W, IC3 B0505S-2W, IC4 B0505S-2W, IC5 1ED3322MC12NXUMA1, J1 Conn_01x02_Male, J10 Conn_01x02_Pin, J11 Conn_01x02_Pin, J12 DC Link Sense, J13 DC Link Sense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

Commit message: Sent gerber to aardra
Parts:
- moved IC4 0.61 mm to (90.1, 131.5)
- moved C17 0.47 mm to (90.6, 121.5)
- moved U3 0.09 mm to (50.9, 161.1)
Connections:
- C5 pad 1: Net-(PS1-CTRL) -> VAux9V
- C6 pad 1: Net-(PS2-CTRL) -> VAux9V
- C8 pad 1: Net-(U3-VO) -> VAux9V
- PS1 pad 2: Net-(PS1-CTRL) -> VAux9V
- PS1 pad 3: Net-(PS1-CTRL) -> VAux9V
- PS2 pad 2: Net-(PS2-CTRL) -> VAux9V
- PS2 pad 3: Net-(PS2-CTRL) -> VAux9V
- U1 pad 3: Net-(PS1-CTRL) -> VAux9V
- U2 pad 3: Net-(PS2-CTRL) -> VAux9V
- U3 pad 3: Net-(U3-VO) -> VAux9V
- U4 pad 3: Net-(U3-VO) -> VAux9V
Routing:
- net VAux9V: track 0.00 -> 51.1 mm
- net Net-(PS1-CTRL): track 32.7 -> 0.00 mm
- net Net-(PS2-CTRL): track 10.1 -> 0.00 mm
- net Net-(U3-VO): track 8.37 -> 0.00 mm
- net VDrive2Neg: track 51.7 -> 52.9 mm
- added copper zone on In1.Cu, net VAux9V
