File: Vegapod 24/Kicad Projects/7.0/Inverter/Inverter/Inverter.kicad_sch (KiCad schematic)
At the start: 122 parts, among them IC1 1ED3322MC12NXUMA1, IC2 B0505S-2W, IC3 B0505S-2W, IC4 B0505S-2W, IC5 1ED3322MC12NXUMA1, J1 Conn_01x02_Male, J10 Conn_01x02_Pin, J11 Conn_01x02_Pin, J12 DC Link Sense, J13 DC Link Sense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

Commit message: Sent gerber to aardra
Connections:
- net VAux9V: now reaches C6.1, PS2.2 (VIN), PS2.3 (CTRL), U2.3 (VO)
- net VAux9V: now also C5.1, C8.1, PS1.2 (VIN), PS1.3 (CTRL), U1.3 (VO), U3.3 (VO), U4.3 (VI)
Changed lines of the file:
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@@
+    )
+  )
+  (global_label "VAux9V" (shape input) (at 87.63 111.76 90) (fields_autoplaced)
+    (effects (font (size 1.27 1.27)) (justify left))
+    (property "Intersheetrefs" "${INTERSHEET_REFS}" (at 87.63 102.1224 90)
+      (effects (font (size 1.27 1.27)) (justify left) hide)
     )
   )
@@
     (effects (font (size 1.27 1.27)) (justify left))
     (property "Intersheetrefs" "${INTERSHEET_REFS}" (at 209.8464 128.1906 0)
+      (effects (font (size 1.27 1.27)) (justify left) hide)
+    )
+  )
+  (global_label "VAux9V" (shape input) (at 69.85 35.56 0) (fields_autoplaced)
+    (effects (font (size 1.27 1.27)) (justify left))
+    (property "Intersheetrefs" "${INTERSHEET_REFS}" (at 79.4876 35.56 0)
       (effects (font (size 1.27 1.27)) (justify left) hide)
     )
@@
       (effects (font (size 1.27 1.27)) (justify left) hide)
     )
+  )
+  (global_label "VAux9V" (shape input) (at 85.09 77.47 90) (fields_autoplaced)
+    (effects (font (size 1.27 1.27)) (justify left))
+    (property "Intersheetrefs" "${INTERSHEET_REFS}" (at 85.09 67.8324 90)
+      (effects (font (size 1.27 1.27)) (justify left) hide)
+    )

Commit message: No changes really
Parts:
- D3: value 1N4007 -> US1M
- D6: value 1N4007 -> US1m
Other:
- moved on the sheet: C29, C3, C36, C37, C4, D20, J12, R10, R29, R30, R31, R32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
