File: Vegapod 24/Kicad Projects/7.0/Chg_Dschg Controller/Chg_Dschg Controller.kicad_pcb (KiCad board)
At the start: 2 copper layers, 85 x 85.1 mm, 47 parts, among them J1 Slave socket, J10 Conn_01x04_Pin, J2 Electronics, J3 Charger, J4 Battery, J5 Contactor, J6 NO/NC Contactor, J7 NC/NO Charge, J8 NO/NC Charge-, J9 NO/NC Charge+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

Commit message: Battery box pcbs done
Routing:
- net Net-(D2-A): track 139.6 -> 138.8 mm
