File: Vegapod 24/Kicad Projects/6.0/LU_Testing/Lu_Testing/Lu_Testing.kicad_sch (KiCad schematic)
At the start: 146 parts, among them J1 DC Link, J2 17V-35V IN, J3 OUT, J4 Conn_01x07_Male, J5 Conn_01x04_Male, J6 Conn_01x04_Male, Q1 Q_NMOS_GDS, Q2 Q_NMOS_GDS, Q3 Q_PMOS_GSD, Q4 Q_PMOS_GSD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

Commit message: Val changes to lu test pcb
Parts:
- C32: value 47n -> 100n
- R46: value Short out -> 1k
Changed lines of the file:
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@@
       (effects (font (size 1.27 1.27)) (justify right))
     )
-    (property "Value" "47n" (id 1) (at 44.45 139.6935 0)
+    (property "Value" "100n" (id 1) (at 44.45 139.6935 0)
       (effects (font (size 1.27 1.27)) (justify right))
     )
@@
   (symbol (lib_id "Device:R") (at -92.71 264.16 0) (unit 1)
     (in_bom yes) (on_board yes) (fields_autoplaced)
-    (property "Reference" "R46" (id 0) (at -90.17 262.8899 0)
+    (property "Reference" "R46" (id 0) (at -88.9 262.8899 0)
       (effects (font (size 1.27 1.27)) (justify left))
     )
-    (property "Value" "Short out" (id 1) (at -90.17 265.4299 0)
+    (property "Value" "1k" (id 1) (at -88.9 265.4299 0)
       (effects (font (size 1.27 1.27)) (justify left))
     )
@@
     )
     (path "/18c25042-dbc9-4119-8029-35b2122f4d3c"
-      (reference "C32") (unit 1) (value "47n") (footprint "Capacitor_SMD:C_0805_2012Metric_Pad1.18x1.45mm_HandSolder")
+      (reference "C32") (unit 1) (value "100n") (footprint "Capacitor_SMD:C_0805_2012Metric_Pad1.18x1.45mm_HandSolder")
     )
     (path "/2ff538ee-c6ba-4efb-89bc-31ed159f75b1"
@@
     )
     (path "/8b05ee23-a4cf-4454-ac48-bef8ce038673"
-      (reference "R46") (unit 1) (value "Short out") (footprint "Resistor_SMD:R_0805_2012Metric_Pad1.20x1.40mm_HandSolder")
+      (reference "R46") (unit 1) (value "1k") (footprint "Resistor_SMD:R_0805_2012Metric_Pad1.20x1.40mm_HandSolder")
     )
     (path "/7845df3c-2f8f-429b-a84d-572d5ca148af"
