File: Vegapod 24/Kicad Projects/7.0/BMS Op/BMS OPAMP/BMS OPAMP.kicad_sch (KiCad schematic)
At the start: 142 parts, among them J1 Balance Connector, J2 NTC1, J3 NTC2, J4 Data IN/OUT, J5 Data IN/OUT, J6 CHG/DSCHG CTRL, J7 Port Selector, J8 Port Selector, J9 CHG/DSCHG CTRL CMP (SHORT DAT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, Q1 MMBT3904, Q2 MMBT3904, Q3 MMBT3904, Q4 MMBT3904, Q5 MMBT3904, Q6 MMBT3904, Q7 MMBT3906, U1 LM324, U10 TLP185, U11 TLP185, U2 LM324, U3 LM324, U4 LM78M05_TO252, U5 TLP185, U6 TLP185, U7 TLP185, U8 6N137, U9 6N137

Commit message: Almost complete bms slave
Parts:
- removed J2: NTC1, Connector_JST:JST_XH_S2B-XH-A_1x02_P2.50mm_Horizontal, symbol Connector:Conn_01x02_Socket
- removed J3: NTC2, Connector_JST:JST_XH_S2B-XH-A_1x02_P2.50mm_Horizontal, symbol Connector:Conn_01x02_Socket
- removed R31, R32: 1k, Resistor_SMD:R_0805_2012Metric_Pad1.20x1.40mm_HandSolder, symbol Device:R
- removed U10, U11, U5, U6, U7: TLP185, Package_SO:SOIC-4_4.55x3.7mm_P2.54mm, symbol Isolator:TLP185
- added J18: Conn_02x06_Odd_Even, Connector_PinSocket_2.00mm:PinSocket_2x06_P2.00mm_Vertical, symbol Connector_Generic:Conn_02x06_Odd_Even
- added J8 (x4): Port Selector, Connector_PinHeader_1.27mm:PinHeader_1x03_P1.27mm_Vertical, symbol Connector:Conn_01x03_Socket
- added Q3 (x3): MMBT3904/AM2304/AO3400, Package_TO_SOT_SMD:SOT-23, symbol Transistor_BJT:MMBT3904
- added R10 (x10), R42 (x6): 47K, Resistor_SMD:R_0805_2012Metric_Pad1.20x1.40mm_HandSolder, symbol Device:R
- added R15 (x3), R43 (x6), R60: 470, Resistor_SMD:R_0805_2012Metric_Pad1.20x1.40mm_HandSolder, symbol Device:R
- added R41, R44 (x5): 33, Resistor_SMD:R_1206_3216Metric_Pad1.30x1.75mm_HandSolder, symbol Device:R
- added R52 (x2): 4.7k, Resistor_SMD:R_0805_2012Metric_Pad1.20x1.40mm_HandSolder, symbol Device:R
- added U1, U12, U2, U3, U4: PC817, Package_SO:SSO-4_6.7x5.1mm_P2.54mm_Clearance8mm, symbol Isolator:PC817
- D1: value 5.1V Z -> Short It Out
- D10, D12, D15, D16, D19, D20: value 1n4007 -> 12V Z
- D11, D13, D14, D17, D18, D9: value 1n4007 -> M7
- J1: footprint Connector_JST:JST_XH_S7B-XH-A_1x07_P2.50mm_Horizontal -> Connector_PinSocket_2.54mm:PinSocket_1x07_P2.54mm_Vertical
- J4: footprint Connector_JST:JST_XH_S3B-XH-A-1_1x03_P2.50mm_Horizontal -> Connector_JST:JST_XH_B3B-XH-A_1x03_P2.50mm_Vertical
- J9: footprint Connector_JST:JST_XH_B6B-XH-AM_1x06_P2.50mm_Vertical -> Connector_PinHeader_2.54mm:PinHeader_1x06_P2.54mm_Vertical
- Q1, Q2, Q3, Q4, Q5, Q6: value MMBT3904 -> MMBT3904/AM2304/AO3400
- Q7: value MMBT3906 -> MMBT3906/FDN358P
- R1, R2, R4: value 10k -> 47k
- R10, R11, R12, R16, R17, R18, R19, R21, R22, R23, R24, R25, R26, R27, R28, R3, R34, R35, R36, R37, R46, R47, R5, R6, R7, R8, R9: value 10k -> 47K
- R13, R14, R15, R20, R29, R30: value 10k -> 470
- R33, R38, R40, R42, R43, R48: value 1k -> 470
- R49: value 1k -> SHORT OUT
- R60: value 330 -> 470
Connections:
- net 5V: now also R52.1, R52.1
- net A6: now also J18.1 (Pin_1), J18.5 (Pin_5), J18.9 (Pin_9), R52.2
- net A7: now also J18.11 (Pin_11), J18.3 (Pin_3), J18.7 (Pin_7), R52.2
- net B0: now also Q3.2 (E), Q3.2 (E), Q3.2 (E), R42.1, U1.3, U12.3, U2.3, U3.2, U4.2
- net B1: now also R10.1, R42.1, R43.1, R44.1; no longer D21.2 (A)
- net B2: now also R10.1, R10.1, R10.1, R10.2, R42.1, R43.1, R44.1; no longer D22.2 (A)
- net B3: now also R10.1, R10.1, R10.1, R10.1, R10.1, R10.1, R10.2, R10.2, R10.2, R41.1, R42.1, R43.1; no longer D26.2 (A)
- net B4: now also R10.2, R10.2, R10.2, R10.2, R10.2, R10.2, R42.1, R43.1, R44.1; no longer D25.2 (A)
- net B5: now also R42.1, R43.1, R44.1; no longer D24.2 (A)
- net B6: now also R43.1, R44.1; no longer D23.2 (A)
- net CHGDT+: now also R60.2
- net CHGDT-: now also U1.2, U2.2
- net DCHG: now also U1.4
- net DIN_GND: now also U12.2
- net at D23.1 (K), Q6.3 (C), R51.2: now also R44.2
- net at J6.4 (Pin_4): now also J8.2 (Pin_2)
- net at J6.6 (Pin_6): now also J8.2 (Pin_2)
- net DTEMP1: now reaches A1.D11 (D11_MOSI)
- net DTEMP1: now also R15.1
- net DTEMP2: now reaches A1.D12 (D12_MISO)
- net DTEMP2: now also R15.1
- net DTEMP3: now reaches A1.D13 (D13_SCK)
- net DTEMP3: now also R15.1
- net at D19.1 (K), Q5.1 (B), R48.2: now also R42.2
- net at D24.1 (K), Q5.3 (C), R50.2: now also R44.2
- net at D16.1 (K), Q4.1 (B), R43.2: now also R42.2
- net at D22.1 (K), Q4.3 (C), R45.2: now also R44.2
- net at D26.1 (K), Q1.3 (C), R39.2: now also R41.2
- net at D21.1 (K), Q3.3 (C), R44.2: now also R44.2
- net at D12.1 (K), Q2.1 (B), R40.2: now also R42.2
- net at R62.2: now also U4.1
- net at R61.1: now also U3.1
- net at D25.1 (K), Q2.3 (C), R41.2: now also R44.2
- net at R52.1: now also U12.4
- net at R53.1: now also U2.4
- net at R60.1: now also U2.1
- net at J9.4 (Pin_4): now also J8.2 (Pin_2)
- net at J9.6 (Pin_6): now also J8.2 (Pin_2)
- net at D20.1 (K), Q6.1 (B), R49.2: now also R42.2
- net at D15.1 (K), Q3.1 (B), R42.2: now also R42.2
- net at R55.1: now also U12.1
- net at D10.1 (K), Q1.1 (B), R38.2: now also R42.2
- new net: J8.1 (Pin_1), J8.1 (Pin_1), U4.3
- new net: J8.3 (Pin_3), J8.3 (Pin_3), U4.4
- new net: D24.2 (A), R43.2
- new net: Q3.1 (B), R15.2 (x3)
- new net: D26.2 (A), R43.2
- new net: J8.1 (Pin_1), J8.1 (Pin_1), U3.3
- new net: J8.3 (Pin_3), J8.3 (Pin_3), U3.4
- new net: D21.2 (A), R43.2
- new net: D22.2 (A), R43.2
- new net: R60.1, U1.1
- new net: D25.2 (A), R43.2
- new net: D23.2 (A), R43.2
- new net NTC_GND1: J18.2 (Pin_2), J18.4 (Pin_4), Q3.3 (C)
- new net NTC_GND2: J18.6 (Pin_6), J18.8 (Pin_8), Q3.3 (C)
- new net NTC_GND3: J18.10 (Pin_10), J18.12 (Pin_12), Q3.3 (C)

Commit message: Almost complete bms slave
Parts:
- removed R10 (x7): 47K, Resistor_SMD:R_0805_2012Metric_Pad1.20x1.40mm_HandSolder, symbol Device:R
- added J6: FTDI, Connector_PinSocket_2.54mm:PinSocket_1x06_P2.54mm_Horizontal, symbol Connector:Conn_01x06_Socket
- added R10: 3.1k, Resistor_SMD:R_0805_2012Metric_Pad1.20x1.40mm_HandSolder, symbol Device:R
- added R10 (x7): 47k, Resistor_SMD:R_0805_2012Metric_Pad1.20x1.40mm_HandSolder, symbol Device:R
- added R10: 4.7K, Resistor_SMD:R_0805_2012Metric_Pad1.20x1.40mm_HandSolder, symbol Device:R
- R10: value 47K -> 47k
Connections:
- net 5V: now also J6.3 (Pin_3)
- net B0: now also J6.1 (Pin_1), J6.2 (Pin_2)
- net B2: now also R10.1, R10.1
- net B3: now also R10.1, R10.1, R10.1, R10.1, R10.1, R10.2, R10.2
- net B4: now also R10.1, R10.2, R10.2, R10.2, R10.2, R10.2
- net B5: now also R10.1, R10.2
- net B6: now also R10.2
- net DRX: now also J6.4 (Pin_4)
- net DTX: now also J6.5 (Pin_5)
- net RST: now reaches A1.RST1 (RESET), A1.RST2 (RESET)
- net RST: now also J6.6 (Pin_6)
Other:
- moved on the sheet: R10

Commit message: BMS PCB
Parts:
- D10, D12, D15, D16, D19, D20: value 12V Z -> 5V Z
Changed lines of the file:
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@@
       (effects (font (size 1.27 1.27)) (justify left))
     )
-    (property "Value" "12V Z" (at 468.63 158.75 90)
+    (property "Value" "5V Z" (at 468.63 158.75 90)
       (effects (font (size 1.27 1.27)) (justify left))
     )
@@
       (effects (font (size 1.27 1.27)) (justify left))
     )
-    (property "Value" "12V Z" (at 576.58 160.02 90)
+    (property "Value" "5V Z" (at 576.58 160.02 90)
       (effects (font (size 1.27 1.27)) (justify left))
     )
@@
       (effects (font (size 1.27 1.27)) (justify left))
     )
-    (property "Value" "12V Z" (at 571.5 43.18 90)
+    (property "Value" "5V Z" (at 571.5 43.18 90)
       (effects (font (size 1.27 1.27)) (justify left))
     )
@@
       (effects (font (size 1.27 1.27)) (justify left))
     )
-    (property "Value" "12V Z" (at 571.5 80.01 90)
+    (property "Value" "5V Z" (at 571.5 80.01 90)
       (effects (font (size 1.27 1.27)) (justify left))
     )
@@
       (effects (font (size 1.27 1.27)) (justify left))
     )
-    (property "Value" "12V Z" (at 467.36 124.46 90)
+    (property "Value" "5V Z" (at 467.36 124.46 90)
       (effects (font (size 1.27 1.27)) (justify left))
     )
@@
       (effects (font (size 1.27 1.27)) (justify left))
     )
-    (property "Value" "12V Z" (at 576.58 123.19 90)
-      (effects (font (size 1.27 1.27)) (justify left))
-    )
+    (property "Value" "5V Z" (at 576.58 123.19 90)
+      (effects (font (size 1.27 1.27)) (justify left))
+    )

Commit message: Minorest change to bms sch
Parts:
- R10: value 3.1k -> 4.7k
Changed lines of the file:
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@@
 (kicad_sch (version 20230121) (generator eeschema)
-  (paper "A4")
+  (paper "A0")
   (junction (at 454.66 73.66) (diameter 0) (color 0 0 0 0)
   )
@@
       (effects (font (size 1.27 1.27)) (justify right))
     )
-    (property "Value" "3.1k" (at 213.36 30.48 0)
+    (property "Value" "4.7k" (at 213.36 30.48 0)
       (effects (font (size 1.27 1.27)) (justify right))
     )
