File: Vegapod 24/Kicad Projects/7.0/Levitation Unit/LU/LU.kicad_sch (KiCad schematic)
At the start: 89 parts, among them IC1 1ED3322MC12NXUMA1, IC2 B0505S-2W, IC3 B0505S-2W, IC4 B0505S-2W, IC5 1ED3322MC12NXUMA1, J1 Conn_01x02_Male, J2 Conn_01x04_Pin, J3 Conn_01x02_Male, Q1 F4-75R06W1E3, U1 LM7809_TO220, U10 6N137, U11 6N137, U2 LM7809_TO220, U3 LM7809_TO220, U4 AMS1117-5.0, U5 AMS1117-5.0, U6 AMS1117-5.0, U8 AMS1117-3.3, U9 ChinaBluePill

Commit message: Levitation Unit completed (review phase)
Parts:
- removed C29: 56uF, Capacitor_THT:CP_Radial_D16.0mm_P7.50mm, symbol Device:C_Polarized
- removed C3, C30, C31, C32, C33, C4: 1000uF, 25V 1000uf:CAP_EEEFK1E102AQ, symbol Device:C_Polarized
- removed C36: 0.1uF, Capacitor_SMD:C_0201_0603Metric_Pad0.64x0.40mm_HandSolder, symbol Device:C
- removed H1, H2, H3, H4: MountingHole, MountingHole:MountingHole_3.2mm_M3, symbol Mechanical:MountingHole
- removed IC2, IC3, IC4: B0505S-2W, B0505-2W:B0505S-2W, symbol B0505S-2W:B0505S-2W
- removed J2: Conn_01x04_Pin, Connector_JST:JST_XH_B4B-XH-AM_1x04_P2.50mm_Vertical, symbol Connector:Conn_01x04_Pin
- removed J3: Conn_01x02_Male, Connector_JST:JST_XH_S2B-XH-A_1x02_P2.50mm_Horizontal, symbol Connector:Conn_01x02_Male
- removed U1, U2, U3: LM7809_TO220, Package_TO_SOT_THT:TO-220-3_Vertical, symbol Regulator_Linear:LM7809_TO220
- removed U10, U11: 6N137, Package_DIP:DIP-8_W7.62mm, symbol Isolator:6N137
- removed U4, U5, U6: AMS1117-5.0, Package_TO_SOT_SMD:SOT-223-3_TabPin2, symbol Regulator_Linear:AMS1117-5.0
- removed U9: ChinaBluePill, BLue Pill:ChinaBluePill, symbol Blue Pill:ChinaBluePill
- added C24, C25, C3, C38, C39, C4: 10uF, Capacitor_SMD:C_1206_3216Metric_Pad1.33x1.80mm_HandSolder, symbol Device:C_Small
- added C29, C32: 1uF 400V, Capacitor_THT:C_Rect_L19.0mm_W9.0mm_P15.00mm_MKS4, symbol Device:C_Small
- added C30, C31: 1uF 400V, Capacitor_THT:C_Rect_L24.0mm_W8.3mm_P22.50mm_MKT, symbol Device:C_Small
- added C33, C36, C37, C40, C42, C43, C45, C48, C51, C53, C55, C57, C60, C62, C63, C64, C65, C66, C67, C70, C71: 100n, Capacitor_SMD:C_0805_2012Metric_Pad1.18x1.45mm_HandSolder, symbol Device:C_Small
- added C41, C44, C46, C49, C52, C54, C56, C58, C59, C61, C68, C69, C72, C73: 10u, Capacitor_SMD:C_1206_3216Metric_Pad1.33x1.80mm_HandSolder, symbol Device:C_Small
- added C47, C50: 10n, Capacitor_SMD:C_0805_2012Metric_Pad1.18x1.45mm_HandSolder, symbol Device:C_Small
- added D7, D8: MUR460, Diode_THT:D_DO-201AE_P15.24mm_Horizontal, symbol Device:D
- added D9: LED, Diode_SMD:D_0805_2012Metric_Pad1.15x1.40mm_HandSolder, symbol Device:LED
- added H6: MountingHole_Pad, MountingHole:MountingHole_6.4mm_M6_DIN965_Pad, symbol Mechanical:MountingHole_Pad
- added H7, H8: MountingHole_Pad, MountingHole:MountingHole_2.2mm_M2_DIN965_Pad, symbol Mechanical:MountingHole_Pad
- added J2: Conn_01x02_Male, Connector_PinSocket_2.54mm:PinSocket_1x02_P2.54mm_Vertical, symbol Connector:Conn_01x02_Male
- added J3: Conn_01x04_Male, Connector_PinHeader_2.54mm:PinHeader_1x04_P2.54mm_Vertical, symbol Connector:Conn_01x04_Male
- added J4: DE9_Receptacle, Connector_Dsub:DSUB-9_Male_Vertical_P2.77x2.84mm, symbol Connector:DE9_Receptacle
- added J5: Conn_01x04_Pin, Connector_PinHeader_1.27mm:PinHeader_1x04_P1.27mm_Vertical, symbol Connector:Conn_01x04_Pin
- added L1, L2, L3, L4, L5, L6, L7: 330uH 5.2A, Inductor_THT:L_Toroid_Vertical_L21.6mm_W11.4mm_P7.62mm_Pulse_KM-3, symbol Device:L
- added PS3: URB2415S-10WR3, URB2415S-10WR3:CONV_URB2415S-10WR3, symbol URB2415S-10WR3:URB2415S-10WR3
- added R26, R57: 50mOhm 3W, Resistor_SMD:R_2512_6332Metric_Pad1.40x3.35mm_HandSolder, symbol Device:R
- added R27, R28, R29, R30, R31, R32: 47, Resistor_SMD:R_0805_2012Metric_Pad1.20x1.40mm_HandSolder, symbol Device:R
- added R33, R34, R35, R36, R41, R53, R61, R62, R63, R64, R65, R66, R70, R72, R73, R74, R75, R76, R77, R78: 470, Resistor_SMD:R_0805_2012Metric_Pad1.20x1.40mm_HandSolder, symbol Device:R
- added R37, R40, R49, R50, R56: 1k, Resistor_SMD:R_0805_2012Metric_Pad1.20x1.40mm_HandSolder, symbol Device:R
- added R38, R39, R51, R52: 47k, Resistor_SMD:R_0805_2012Metric_Pad1.20x1.40mm_HandSolder, symbol Device:R
- added R42, R54: SHORT OUT, Resistor_SMD:R_0805_2012Metric_Pad1.20x1.40mm_HandSolder, symbol Device:R
- added R43, R55: OPEN CIRCUIT, Resistor_SMD:R_0805_2012Metric_Pad1.20x1.40mm_HandSolder, symbol Device:R
- added R44, R46: 22k, Resistor_SMD:R_0805_2012Metric_Pad1.20x1.40mm_HandSolder, symbol Device:R
- added R45, R47: 22K, Resistor_SMD:R_0805_2012Metric_Pad1.20x1.40mm_HandSolder, symbol Device:R
- added R48: 1K, Resistor_SMD:R_0805_2012Metric_Pad1.20x1.40mm_HandSolder, symbol Device:R
- added R5, R58, R6: 1R, Resistor_SMD:R_0805_2012Metric_Pad1.20x1.40mm_HandSolder, symbol Device:R
- added R59: SHORT OUT, Resistor_SMD:R_0402_1005Metric, symbol Device:R
- added R60: Open Circuit, Resistor_SMD:R_0402_1005Metric, symbol Device:R
- added R67, R68, R69, R71: 10k, Resistor_SMD:R_0805_2012Metric_Pad1.20x1.40mm_HandSolder, symbol Device:R
- added U1, U2, U5: 78m09, Package_TO_SOT_SMD:TO-252-2, symbol Regulator_Linear:KA78M05_TO252
- added U10, U11, U12, U9: ADUM4195-1BRIZ, RI-8-1_ADI, symbol ADUM-4195:ADUM4195-1BRIZ
- added U13, U6: LM324, Package_SO:SOIC-14_3.9x8.7mm_P1.27mm, symbol Amplifier_Operational:LM324
- added U14: STM32G474RETx, Package_QFP:LQFP-64_10x10mm_P0.5mm, symbol MCU_ST_STM32G4:STM32G474RETx
- added U15, U16: 6N137, Package_SO:SSO-8_6.7x9.8mm_P2.54mm_Clearance8mm, symbol Isolator:6N137
- added U3: KA78M05_TO252, Package_TO_SOT_SMD:TO-252-2, symbol Regulator_Linear:KA78M05_TO252
- added U4: B0505S-1WR3, B0505S_MNS, symbol B0505-1WR3:B0505S-1WR3
- added U7: AMS1117-5.0, Package_TO_SOT_SMD:SOT-223-3_TabPin2, symbol Regulator_Linear:AMS1117-5.0
- C1, C10, C11, C12, C14, C15, C16, C18, C19, C2, C21, C22, C6, C7, C8, C9: value 1uF -> 10uF
- C13, C5: value 1uF -> 100n; footprint Capacitor_SMD:C_1206_3216Metric_Pad1.33x1.80mm_HandSolder -> Capacitor_SMD:C_0805_2012Metric_Pad1.18x1.45mm_HandSolder
- C17: value 1uF -> 100nF; footprint Capacitor_SMD:C_1206_3216Metric_Pad1.33x1.80mm_HandSolder -> Capacitor_SMD:C_0805_2012Metric_Pad1.18x1.45mm_HandSolder
- C26: value 22nF -> 1uF
- C27, C28: value 22nF -> C_Snub 1uF 400V; footprint Capacitor_SMD:C_1206_3216Metric_Pad1.33x1.80mm_HandSolder -> Capacitor_THT:C_Rect_L24.0mm_W8.3mm_P22.50mm_MKT
- D3, D6: value 1N4007 -> US1M
- H5: value Output - -> MountingHole_Pad; footprint MountingHole:MountingHole_6.4mm_M6_Pad -> MountingHole:MountingHole_6.4mm_M6_DIN965_Pad
- J1: footprint Connector_JST:JST_XH_S2B-XH-A_1x02_P2.50mm_Horizontal -> Connector_JST:JST_XH_B2B-XH-A_1x02_P2.50mm_Vertical
- R1, R3: value 3.3 -> 1R
- R11, R12, R13, R14, R15, R17, R18, R19, R20: value 1 -> 50mOhm 3W
- R16: value 1 -> R_Snub 220Ohm 1W; footprint Resistor_SMD:R_2512_6332Metric_Pad1.40x3.35mm_HandSolder -> Resistor_THT:R_Box_L26.0mm_W5.0mm_P20.00mm
- R21, R23, R24, R25: value 330 -> 50mOhm 3W; footprint Resistor_SMD:R_0201_0603Metric_Pad0.64x0.40mm_HandSolder -> Resistor_SMD:R_2512_6332Metric_Pad1.40x3.35mm_HandSolder
- R22: value 470 -> 50mOhm 3W; footprint Resistor_SMD:R_0201_0603Metric_Pad0.64x0.40mm_HandSolder -> Resistor_SMD:R_2512_6332Metric_Pad1.40x3.35mm_HandSolder
- R7: value 22K -> R_Snub 220Ohm 1W; footprint Resistor_SMD:R_1206_3216Metric_Pad1.30x1.75mm_HandSolder -> Resistor_THT:R_Box_L26.0mm_W5.0mm_P20.00mm
Connections:
- net +BATT: now also Q1.P1, Q1.P2, Q1.P3, R7.2, C30.2, C31.2, D9.2 (A), H6.1, R44.1; no longer C26.1, C28.1, R7.1
- net -BATT: now also Q1.EU1, Q1.EU2, Q1.EU3, Q1.EV1, Q1.EV2, Q1.EV3, R17.2, R18.2, R19.2, R20.2, R21.2, R22.2, R23.2, R24.2, R25.2, C29.1, C30.1, C31.1, C32.1, R26.2, R32.2, R35.2, R57.1, R68.2; no longer C14.2, C15.2, C27.2, C34.2, C35.2, IC1.11 (IN-), IC1.16 (GND1_2), IC1.9 (GND1_1), IC5.11 (IN-), IC5.16 (GND1_2), IC5.9 (GND1_1), R10.1, R17.1, R18.1, R19.1, R20.1, R22.1, R7.2, U8.1 (GND)
- net DIG+: now also C18.1, C22.1, C60.2, C61.2, C62.2, C63.2, C64.2, C65.2, C72.1, J4.2, J5.1 (Pin_1), R58.2, R60.2, U14.1 (VBAT), U14.16 (VDD), U14.32 (VDD), U14.48 (VDD), U14.64 (VDD)
- net DIG5V: now also C51.2, C52.2, C53.2, C54.2, C55.2, C56.2, C57.2, C58.2, C59.2, C70.2, C73.1, J4.3, R61.1, R62.1, U10.8 (VDD1), U11.8 (VDD1), U12.8 (VDD1), U13.4 (V+), U15.7 (EN), U15.8 (VCC), U4.4 (+VO), U9.8 (VDD1); no longer R21.2
- net GND1: now also C20.2, D2.2 (A), IC1.1 (VEE2_1), IC1.8 (VEE2_2), Q1.E2, Q1.E4; no longer C16.1, C18.1
- net GND2: now also C23.2, D5.2 (A), IC5.1 (VEE2_1), IC5.8 (VEE2_2), Q1.E1, Q1.E3, C24.2; no longer C13.2, C17.1, C22.1
- net INHS: now also U14.8 (PC0)
- net INLS: now also U14.2 (PC13)
- net VAux+: now also C8.1, J2.2 (Pin_2), U1.1 (VI), U2.1 (VI), U3.1 (VI), U5.1 (VI)
- net VAux-: now also C25.2, C3.2, J2.1 (Pin_1), PS3.1 (GND), U1.2 (GND), U2.2 (GND), U3.2 (GND), U4.1 (GND), U5.2 (GND); no longer C5.2
- net VDrive1: now also C12.1
- net VDrive2: now also C24.1
- net DCLink-: now reaches H5.1, R11.2, R12.2, R13.2, R14.2, R15.2
- net DCLink-: now also C16.2, C17.2, C26.1, C38.2, C39.2, C4.2, C40.1, C41.1, C42.1, C43.1, C44.1, C45.1, C46.1, C47.1, C48.1, C49.1, C50.1, PS3.7 (0V), R36.2, R38.2, R41.2, R43.2, R48.2, R51.2, R53.2, R55.2, R56.1, R57.2, U10.3 (SHTD), U10.4 (GND2), U11.3 (SHTD), U11.4 (GND2), U12.3 (SHTD), U12.4 (GND2), U6.11 (V-), U7.1 (GND), U9.3 (SHTD), U9.4 (GND2); no longer R16.2, R17.2, R18.2, R19.2, R20.2
- net at C6.1, PS2.2 (VIN), PS2.3 (CTRL): now also U1.3 (VO)
- net at C11.1: now also U3.3 (VO), U4.2 (VIN)
- net OUT-: now reaches R24.1
- net OUT-: now also R17.1, R18.1, R19.1, R20.1, R21.1, R22.1, R23.1, R25.1, H7.1, R26.1, R29.2
- net at C13.1: now also R34.2, R36.1
- net at PS1.2 (VIN), PS1.3 (CTRL): now also C25.1, U2.3 (VO); no longer C5.1
- net at IC5.4 (OUT-): now also R6.1
- net at IC5.7 (CLAMP): now also Q1.G1, Q1.G3, R3.2, R6.2
- net at R1.2: now also IC1.7 (CLAMP), Q1.G2, Q1.G4, R5.2
- net SensePWR5V: now reaches Q1.T2
- net SensePWR5V: now also C39.1, C40.2, C41.2, C43.2, C44.2, C45.2, C46.2, C48.2, C49.2, U10.1 (VDD2), U11.1 (VDD2), U12.1 (VDD2), U7.2 (VO), U9.1 (VDD2); no longer Q1.T1
- net at Q1.U1, Q1.U2, Q1.U3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: now also D7.1 (K), D8.2 (A), L1.1, L2.1, L3.1, L4.1, L5.1, L6.1, L7.1
- net at IC1.4 (OUT-): now also R5.1
- removed net VDrive1Neg: C16.2, C18.2, C20.2, D2.2 (A), IC1.1 (VEE2_1), IC1.8 (VEE2_2)
- removed net VDrive2Neg: C17.2, C22.2, C23.2, D5.2 (A), IC5.1 (VEE2_1), IC5.8 (VEE2_2)
- new net: R75.2, U12.7 (VOUT), U13.12 (+)
- new net: C3.1, PS3.2 (VIN), PS3.3 (CTRL), U5.3 (VO)
- new net: R62.2, R63.2, U16.2 (A)
- new net: R37.2, R38.1, U6.3 (+)
- new net: R65.1, R66.1, U15.2 (A)
- new net: R76.2, U11.7 (VOUT), U13.10 (+)
- new net: R77.2, U10.7 (VOUT), U13.5 (+)
- new net: R45.2, R46.1
- new net: R46.2, R47.1
- new net: C36.1, R30.2, R31.1
- new net: C36.2, R27.2, R28.1
- new net: C67.1, U14.7 (PG10)
- new net: R49.2, R51.1, U6.10 (+)
- new net: C37.2, R28.2, R29.1
- new net: R59.2, R60.1, U14.61 (PB8)
- new net: R52.1, R53.1, R54.1, U6.8
- new net: R50.2, R52.2, U6.9 (-)
- new net: R39.1, R41.1, R42.1, U6.1
- new net: C66.1, C68.1, R58.1, U14.28 (VREF+), U14.29 (VDDA)
- new net: C27.2, D7.2 (A), R16.2
- new net: R39.2, R40.2, U6.2 (-)
- new net: R44.2, R45.1
- new net: R67.1, R68.1
- new net: C37.1, R31.2, R32.1
- new net: R78.2, U13.3 (+), U9.7 (VOUT)
- new net: C13.2, R33.2, R35.1
- new net: C28.1, D8.1 (K), R7.1
- new net: R67.2, R69.1
- new net: R69.2, R71.1
- new net: D9.1 (K), R71.2
- new net: PS3.5 (NC), PS3.8 (NC)
- new net 5VCOMM: C69.2, C71.2, J3.4 (Pin_4), R64.2, R65.2, U16.7 (EN), U16.8 (VCC)
- new net A0: C47.2, R42.2, R43.1, U11.2 (VIN)
- new net A1: C17.1, R47.2, R48.1, U10.2 (VIN)
- new net A2: C50.2, R54.2, R55.1, U12.2 (VIN)
- new net DA0: R74.1, U13.1, U13.2 (-), U14.42 (PA8)
- new net DA1: R73.1, U13.6 (-), U13.7, U14.25 (PB1)
- new net DA2: R70.1, U13.8, U13.9 (-), U14.12 (PA0)
- new net DA3: R72.1, U13.13 (-), U13.14, U14.34 (PB12)
- new net DIG-: C14.2, C15.2, C18.2, C22.2, C34.2, C35.2, C51.1, C52.1, C53.1, C54.1, C55.1, C56.1, C57.1, C58.1, C59.1, C60.1, C61.1, C62.1, C63.1, C64.1, C65.1, C66.2, C67.2, C68.2, C70.1, C72.2, C73.2, IC1.11 (IN-), IC1.16 (GND1_2), IC1.9 (GND1_1), IC5.11 (IN-), IC5.16 (GND1_2), IC5.9 (GND1_1), J4.1, J5.4 (Pin_4), R10.1, R59.1, R63.1, R70.2, R72.2, R73.2, R74.2, R75.1, R76.1, R77.1, R78.1, U10.5 (GND1), U10.6 (NC), U11.5 (GND1), U11.6 (NC), U12.5 (GND1), U12.6 (NC), U13.11 (V-), U14.15 (VSS), U14.27 (VSSA), U14.31 (VSS), U14.47 (VSS), U14.63 (VSS), U15.5 (GND), U4.3 (0V), U8.1 (GND), U9.5 (GND1), U9.6 (NC)
- new net GNDCOMM: C69.1, C71.1, J3.1 (Pin_1), R66.2, U16.5 (GND)
- new net INSHUNT+: C5.2, R33.1, R49.1
- new net INSHUNT-: C5.1, R34.1, R50.1
- new net OUT+: C29.2, C32.2, H8.1, L1.2, L2.2, L3.2, L4.2, L5.2, L6.2, L7.2
- new net OUTSHUNT+: C33.2, R27.1, R37.1
- new net OUTSHUNT-: C33.1, R30.1, R40.1
- new net RXCOMM: J3.2 (Pin_2), U15.3 (C)
- new net RXD: J4.4, R61.2, U14.23 (PC5), U15.6 (VO)
- new net SWCLK: J4.6, J5.2 (Pin_2), U14.50 (PA14)
- new net SWDIO: J4.7, J5.3 (Pin_3), U14.49 (PA13)
- new net SensePWR: C16.1, C38.1, C4.1, PS3.6 (+VO), U6.4 (V+), U7.3 (VI)
- new net T-: C42.2, Q1.T1, R56.2, U9.2 (VIN)
- new net TXCOMM: J3.3 (Pin_3), R64.1, U16.6 (VO)
- new net TXD: J4.5, U14.22 (PC4), U16.3 (C)
- no-connect marks 2 -> 0
