File: Vegapod 24/Kicad Projects/7.0/Levitation Unit/LU/LU.kicad_pcb (KiCad board)
At the start: 2 copper layers, 96 parts, among them IC1 1ED3322MC12NXUMA1, IC2 B0505S-2W, IC3 B0505S-2W, IC4 B0505S-2W, IC5 1ED3322MC12NXUMA1, J1 Conn_01x02_Male, J2 Conn_01x04_Pin, J3 Conn_01x02_Male, Q1 F4-75R06W1E3, U1 LM7809_TO220, U10 6N137, U11 6N137, U2 LM7809_TO220, U3 LM7809_TO220, U4 AMS1117-5.0, U5 AMS1117-5.0, U6 AMS1117-5.0, U7 FF150R12RT4, U8 AMS1117-3.3, U9 ChinaBluePill

Commit message: Levitation Unit completed (review phase)
Parts:
- removed H1, H2, H3, H4: MountingHole, MountingHole:MountingHole_3.2mm_M3
- removed IC2, IC3, IC4: B0505S-2W, B0505-2W:B0505S-2W
- added C37: 100n, Capacitor_SMD:C_0805_2012Metric_Pad1.18x1.45mm_HandSolder, F.Cu at (211.0, 190.0)
- added C38: 10uF, Capacitor_SMD:C_1206_3216Metric_Pad1.33x1.80mm_HandSolder, F.Cu at (114.8, 186.0)
- added C39: 10uF, Capacitor_SMD:C_1206_3216Metric_Pad1.33x1.80mm_HandSolder, B.Cu at (117.0, 178.5)
- added C40: 100n, Capacitor_SMD:C_0805_2012Metric_Pad1.18x1.45mm_HandSolder, B.Cu at (124.8, 159.5)
- added C41: 10u, Capacitor_SMD:C_1206_3216Metric_Pad1.33x1.80mm_HandSolder, B.Cu at (122.5, 160.2)
- added C42: 100n, Capacitor_SMD:C_0805_2012Metric_Pad1.18x1.45mm_HandSolder, F.Cu at (129.0, 159.5)
- added C43: 100n, Capacitor_SMD:C_0805_2012Metric_Pad1.18x1.45mm_HandSolder, B.Cu at (124.8, 166.0)
- added C44: 10u, Capacitor_SMD:C_1206_3216Metric_Pad1.33x1.80mm_HandSolder, B.Cu at (122.5, 166.8)
- added C45: 100n, Capacitor_SMD:C_0805_2012Metric_Pad1.18x1.45mm_HandSolder, B.Cu at (124.8, 173.0)
- added C46: 10u, Capacitor_SMD:C_1206_3216Metric_Pad1.33x1.80mm_HandSolder, B.Cu at (122.5, 173.5)
- added C47: 10n, Capacitor_SMD:C_0805_2012Metric_Pad1.18x1.45mm_HandSolder, F.Cu at (129.2, 173.0)
- added C48: 100n, Capacitor_SMD:C_0805_2012Metric_Pad1.18x1.45mm_HandSolder, F.Cu at (124.5, 181.2)
- added C49: 10u, Capacitor_SMD:C_1206_3216Metric_Pad1.33x1.80mm_HandSolder, F.Cu at (126.8, 180.5)
- added C50: 10n, Capacitor_SMD:C_0805_2012Metric_Pad1.18x1.45mm_HandSolder, B.Cu at (122.8, 179.8)
- added C51: 100n, Capacitor_SMD:C_0805_2012Metric_Pad1.18x1.45mm_HandSolder, F.Cu at (114.8, 160.2)
- added C52: 10u, Capacitor_SMD:C_1206_3216Metric_Pad1.33x1.80mm_HandSolder, B.Cu at (114.8, 159.8)
- added C53: 100n, Capacitor_SMD:C_0805_2012Metric_Pad1.18x1.45mm_HandSolder, F.Cu at (114.8, 167.2)
- added C54: 10u, Capacitor_SMD:C_1206_3216Metric_Pad1.33x1.80mm_HandSolder, B.Cu at (114.8, 166.8)
- added C55: 100n, Capacitor_SMD:C_0805_2012Metric_Pad1.18x1.45mm_HandSolder, F.Cu at (114.8, 174.0)
- added C56: 10u, Capacitor_SMD:C_1206_3216Metric_Pad1.33x1.80mm_HandSolder, B.Cu at (114.8, 173.5)
- added C57: 100n, Capacitor_SMD:C_0805_2012Metric_Pad1.18x1.45mm_HandSolder, F.Cu at (110.0, 181.2)
- added C58: 10u, Capacitor_SMD:C_1206_3216Metric_Pad1.33x1.80mm_HandSolder, B.Cu at (110.0, 180.8)
- added C59: 10u, Capacitor_SMD:C_1206_3216Metric_Pad1.33x1.80mm_HandSolder, B.Cu at (103.1, 184.5)
- added C60: 100n, Capacitor_SMD:C_0805_2012Metric_Pad1.18x1.45mm_HandSolder, B.Cu at (103.0, 161.8)
- added C61: 10u, Capacitor_SMD:C_1206_3216Metric_Pad1.33x1.80mm_HandSolder, B.Cu at (103.5, 157.5)
- added C62: 100n, Capacitor_SMD:C_0805_2012Metric_Pad1.18x1.45mm_HandSolder, B.Cu at (100.0, 163.0)
- added C63: 100n, Capacitor_SMD:C_0805_2012Metric_Pad1.18x1.45mm_HandSolder, B.Cu at (99.2, 168.8)
- added C64: 100n, Capacitor_SMD:C_0805_2012Metric_Pad1.18x1.45mm_HandSolder, F.Cu at (110.2, 172.8)
- added C65: 100n, Capacitor_SMD:C_0805_2012Metric_Pad1.18x1.45mm_HandSolder, B.Cu at (108.8, 162.8)
- added C66: 100n, Capacitor_SMD:C_0805_2012Metric_Pad1.18x1.45mm_HandSolder, B.Cu at (108.5, 170.8)
- added C67: 100n, Capacitor_SMD:C_0805_2012Metric_Pad1.18x1.45mm_HandSolder, B.Cu at (101.3, 166.8)
- added C68: 10u, Capacitor_SMD:C_1206_3216Metric_Pad1.33x1.80mm_HandSolder, B.Cu at (106.2, 171.5)
- added C69: 10u, Capacitor_SMD:C_1206_3216Metric_Pad1.33x1.80mm_HandSolder, B.Cu at (113.0, 97.5)
- added C70: 100n, Capacitor_SMD:C_0805_2012Metric_Pad1.18x1.45mm_HandSolder, B.Cu at (112.8, 107.0)
- added C71: 100n, Capacitor_SMD:C_0805_2012Metric_Pad1.18x1.45mm_HandSolder, F.Cu at (99.8, 96.0)
- added C72: 10u, Capacitor_SMD:C_1206_3216Metric_Pad1.33x1.80mm_HandSolder, B.Cu at (103.4, 132.7)
- added C73: 10u, Capacitor_SMD:C_1206_3216Metric_Pad1.33x1.80mm_HandSolder, B.Cu at (103.5, 148.0)
- added D9: LED, Diode_SMD:D_0805_2012Metric_Pad1.15x1.40mm_HandSolder, F.Cu at (167.0, 171.2)
- added H6: MountingHole_Pad, MountingHole:MountingHole_6.4mm_M6_DIN965_Pad, F.Cu at (145.0, 188.5)
- added H7: MountingHole_Pad, MountingHole:MountingHole_2.2mm_M2_DIN965_Pad, F.Cu at (213.0, 151.5)
- added H8: MountingHole_Pad, MountingHole:MountingHole_2.2mm_M2_DIN965_Pad, F.Cu at (213.0, 142.0)
- added J4: DE9_Receptacle, Connector_Dsub:DSUB-9_Male_Vertical_P2.77x2.84mm, F.Cu at (104.8, 134.8)
- added J5: Conn_01x04_Pin, Connector_PinHeader_1.27mm:PinHeader_1x04_P1.27mm_Vertical, B.Cu at (105.6, 125.5)
- added L1: 330uH 5.2A, Inductor_THT:L_Toroid_Vertical_L21.6mm_W11.4mm_P7.62mm_Pulse_KM-3, F.Cu at (196.0, 97.8)
- added L2: 330uH 5.2A, Inductor_THT:L_Toroid_Vertical_L21.6mm_W11.4mm_P7.62mm_Pulse_KM-3, F.Cu at (196.0, 110.8)
- added L3: 330uH 5.2A, Inductor_THT:L_Toroid_Vertical_L21.6mm_W11.4mm_P7.62mm_Pulse_KM-3, F.Cu at (196.0, 123.8)
- added L4: 330uH 5.2A, Inductor_THT:L_Toroid_Vertical_L21.6mm_W11.4mm_P7.62mm_Pulse_KM-3, F.Cu at (196.0, 136.8)
- added L5: 330uH 5.2A, Inductor_THT:L_Toroid_Vertical_L21.6mm_W11.4mm_P7.62mm_Pulse_KM-3, F.Cu at (195.9, 149.8)
- added L6: 330uH 5.2A, Inductor_THT:L_Toroid_Vertical_L21.6mm_W11.4mm_P7.62mm_Pulse_KM-3, F.Cu at (195.9, 162.7)
- added L7: 330uH 5.2A, Inductor_THT:L_Toroid_Vertical_L21.6mm_W11.4mm_P7.62mm_Pulse_KM-3, F.Cu at (195.9, 175.7)
- added PS3: URB2415S-10WR3, URB2415S-10WR3:CONV_URB2415S-10WR3, F.Cu at (109.3, 192.3)
- added R26: 50mOhm 3W, Resistor_SMD:R_2512_6332Metric_Pad1.40x3.35mm_HandSolder, B.Cu at (211.0, 192.0)
- added R27: 47, Resistor_SMD:R_0805_2012Metric_Pad1.20x1.40mm_HandSolder, F.Cu at (214.2, 194.0)
- added R28: 47, Resistor_SMD:R_0805_2012Metric_Pad1.20x1.40mm_HandSolder, F.Cu at (213.0, 192.0)
- added R29: 47, Resistor_SMD:R_0805_2012Metric_Pad1.20x1.40mm_HandSolder, F.Cu at (213.0, 188.0)
- added R30: 47, Resistor_SMD:R_0805_2012Metric_Pad1.20x1.40mm_HandSolder, F.Cu at (206.6, 194.0)
- added R31: 47, Resistor_SMD:R_0805_2012Metric_Pad1.20x1.40mm_HandSolder, F.Cu at (209.0, 192.0)
- added R32: 47, Resistor_SMD:R_0805_2012Metric_Pad1.20x1.40mm_HandSolder, F.Cu at (209.0, 188.0)
- added R33: 470, Resistor_SMD:R_0805_2012Metric_Pad1.20x1.40mm_HandSolder, B.Cu at (129.6, 177.5)
- added R34: 470, Resistor_SMD:R_0805_2012Metric_Pad1.20x1.40mm_HandSolder, B.Cu at (129.7, 179.6)
- added R35: 470, Resistor_SMD:R_0805_2012Metric_Pad1.20x1.40mm_HandSolder, B.Cu at (135.7, 177.1)
- added R36: 470, Resistor_SMD:R_0805_2012Metric_Pad1.20x1.40mm_HandSolder, B.Cu at (135.8, 180.3)
- added R37: 1k, Resistor_SMD:R_0805_2012Metric_Pad1.20x1.40mm_HandSolder, B.Cu at (130.8, 195.8)
- added R38: 47k, Resistor_SMD:R_0805_2012Metric_Pad1.20x1.40mm_HandSolder, B.Cu at (127.8, 194.9)
- added R39: 47k, Resistor_SMD:R_0805_2012Metric_Pad1.20x1.40mm_HandSolder, F.Cu at (133.9, 192.7)
- added R40: 1k, Resistor_SMD:R_0805_2012Metric_Pad1.20x1.40mm_HandSolder, B.Cu at (132.9, 196.0)
- added R41: 470, Resistor_SMD:R_0805_2012Metric_Pad1.20x1.40mm_HandSolder, B.Cu at (135.8, 194.8)
- added R42: SHORT OUT, Resistor_SMD:R_0805_2012Metric_Pad1.20x1.40mm_HandSolder, F.Cu at (130.0, 191.7)
- added R43: OPEN CIRCUIT, Resistor_SMD:R_0805_2012Metric_Pad1.20x1.40mm_HandSolder, F.Cu at (130.0, 193.7)
- added R44: 22k, Resistor_SMD:R_0805_2012Metric_Pad1.20x1.40mm_HandSolder, F.Cu at (136.1, 158.7)
- added R45: 22K, Resistor_SMD:R_0805_2012Metric_Pad1.20x1.40mm_HandSolder, F.Cu at (135.7, 160.7)
- added R46: 22k, Resistor_SMD:R_0805_2012Metric_Pad1.20x1.40mm_HandSolder, F.Cu at (135.7, 162.8)
- added R47: 22K, Resistor_SMD:R_0805_2012Metric_Pad1.20x1.40mm_HandSolder, F.Cu at (135.7, 165.0)
- added R48: 1K, Resistor_SMD:R_0805_2012Metric_Pad1.20x1.40mm_HandSolder, F.Cu at (136.5, 168.1)
- added R49: 1k, Resistor_SMD:R_0805_2012Metric_Pad1.20x1.40mm_HandSolder, B.Cu at (129.7, 182.8)
- added R50: 1k, Resistor_SMD:R_0805_2012Metric_Pad1.20x1.40mm_HandSolder, B.Cu at (127.7, 182.7)
- added R51: 47k, Resistor_SMD:R_0805_2012Metric_Pad1.20x1.40mm_HandSolder, B.Cu at (132.6, 183.8)
- added R52: 47k, Resistor_SMD:R_0805_2012Metric_Pad1.20x1.40mm_HandSolder, B.Cu at (125.6, 182.7)
- added R53: 470, Resistor_SMD:R_0805_2012Metric_Pad1.20x1.40mm_HandSolder, B.Cu at (123.3, 186.2)
- added R54: SHORT OUT, Resistor_SMD:R_0805_2012Metric_Pad1.20x1.40mm_HandSolder, B.Cu at (122.6, 184.1)
- added R55: OPEN CIRCUIT, Resistor_SMD:R_0805_2012Metric_Pad1.20x1.40mm_HandSolder, B.Cu at (122.7, 182.0)
- added R56: 1k, Resistor_SMD:R_0805_2012Metric_Pad1.20x1.40mm_HandSolder, F.Cu at (131.0, 159.5)
- added R57: 50mOhm 3W, Resistor_SMD:R_2512_6332Metric_Pad1.40x3.35mm_HandSolder, B.Cu at (163.2, 177.0)
- added R58: 1R, Resistor_SMD:R_0805_2012Metric_Pad1.20x1.40mm_HandSolder, F.Cu at (107.2, 174.4)
- added R59: SHORT OUT, Resistor_SMD:R_0402_1005Metric, F.Cu at (103.2, 157.5)
- added R60: Open Circuit, Resistor_SMD:R_0402_1005Metric, F.Cu at (102.2, 157.5)
- added R61: 470, Resistor_SMD:R_0805_2012Metric_Pad1.20x1.40mm_HandSolder, F.Cu at (112.8, 107.0)
- added R62: 470, Resistor_SMD:R_0805_2012Metric_Pad1.20x1.40mm_HandSolder, F.Cu at (100.4, 106.2)
- added R63: 470, Resistor_SMD:R_0805_2012Metric_Pad1.20x1.40mm_HandSolder, F.Cu at (98.5, 106.2)
- added R64: 470, Resistor_SMD:R_0805_2012Metric_Pad1.20x1.40mm_HandSolder, F.Cu at (113.2, 97.0)
- added R65: 470, Resistor_SMD:R_0805_2012Metric_Pad1.20x1.40mm_HandSolder, B.Cu at (99.4, 97.0)
- added R66: 470, Resistor_SMD:R_0805_2012Metric_Pad1.20x1.40mm_HandSolder, B.Cu at (99.4, 95.0)
- added R67: 10k, Resistor_SMD:R_0805_2012Metric_Pad1.20x1.40mm_HandSolder, F.Cu at (167.0, 177.6)
- added R68: 10k, Resistor_SMD:R_0805_2012Metric_Pad1.20x1.40mm_HandSolder, F.Cu at (168.6, 179.8)
- added R69: 10k, Resistor_SMD:R_0805_2012Metric_Pad1.20x1.40mm_HandSolder, F.Cu at (167.0, 175.4)
- added R70: 470, Resistor_SMD:R_0805_2012Metric_Pad1.20x1.40mm_HandSolder, B.Cu at (103.6, 172.0)
- added R71: 10k, Resistor_SMD:R_0805_2012Metric_Pad1.20x1.40mm_HandSolder, F.Cu at (167.0, 173.2)
- added R72: 470, Resistor_SMD:R_0805_2012Metric_Pad1.20x1.40mm_HandSolder, B.Cu at (107.8, 182.8)
- added R73: 470, Resistor_SMD:R_0805_2012Metric_Pad1.20x1.40mm_HandSolder, B.Cu at (98.2, 176.0)
- added R74: 470, Resistor_SMD:R_0805_2012Metric_Pad1.20x1.40mm_HandSolder, B.Cu at (98.2, 183.0)
- added R75: 470, Resistor_SMD:R_0805_2012Metric_Pad1.20x1.40mm_HandSolder, F.Cu at (105.4, 182.0)
- added R76: 470, Resistor_SMD:R_0805_2012Metric_Pad1.20x1.40mm_HandSolder, B.Cu at (118.4, 172.0)
- added R77: 470, Resistor_SMD:R_0805_2012Metric_Pad1.20x1.40mm_HandSolder, B.Cu at (118.4, 165.2)
- added R78: 470, Resistor_SMD:R_0805_2012Metric_Pad1.20x1.40mm_HandSolder, B.Cu at (118.4, 158.2)
- added U12: ADUM4195-1BRIZ, ADUM-4195:RI-8-1_ADI, F.Cu at (117.2, 180.8)
- added U13: LM324, Package_SO:SOIC-14_3.9x8.7mm_P1.27mm, B.Cu at (103.0, 178.7)
- added U14: STM32G474RETx, Package_QFP:LQFP-64_10x10mm_P0.5mm, F.Cu at (104.5, 165.5)
- added U15: 6N137, Package_SO:SSO-8_6.7x9.8mm_P2.54mm_Clearance8mm, B.Cu at (106.6, 103.3)
- added U16: 6N137, Package_SO:SSO-8_6.7x9.8mm_P2.54mm_Clearance8mm, F.Cu at (106.6, 103.5)
- C1, C10, C11, C12, C14, C16, C18, C19, C2, C21, C22, C6, C7, C8: value 1uF -> 10uF; moved to B.Cu
- C13, C5: value 1uF -> 100n; footprint Capacitor_SMD:C_1206_3216Metric_Pad1.33x1.80mm_HandSolder -> Capacitor_SMD:C_0805_2012Metric_Pad1.18x1.45mm_HandSolder; moved to B.Cu
- C15, C9: value 1uF -> 10uF
- C17: value 1uF -> 100nF; footprint Capacitor_SMD:C_1206_3216Metric_Pad1.33x1.80mm_HandSolder -> Capacitor_SMD:C_0805_2012Metric_Pad1.18x1.45mm_HandSolder
- C20, C23, C34, C35, D1, D2, D4, D5, Q1, R2, R4, R8, U8: moved to B.Cu
- C24: value C_Snub -> 10uF; footprint Capacitor_THT:C_Rect_L24.0mm_W8.3mm_P22.50mm_MKT -> Capacitor_SMD:C_1206_3216Metric_Pad1.33x1.80mm_HandSolder
- C25: value C_Snub -> 10uF; footprint Capacitor_THT:C_Rect_L24.0mm_W8.3mm_P22.50mm_MKT -> Capacitor_SMD:C_1206_3216Metric_Pad1.33x1.80mm_HandSolder; moved to B.Cu
- C26: value 22nF -> 1uF; moved to B.Cu
- C27, C28: value 22nF -> C_Snub 1uF 400V; footprint Capacitor_SMD:C_1206_3216Metric_Pad1.33x1.80mm_HandSolder -> Capacitor_THT:C_Rect_L24.0mm_W8.3mm_P22.50mm_MKT
- C29: value 56uF -> 1uF 400V; footprint Capacitor_THT:CP_Radial_D16.0mm_P7.50mm -> Capacitor_THT:C_Rect_L19.0mm_W9.0mm_P15.00mm_MKS4
- C3, C4: value 1000uF -> 10uF; footprint 25V 1000uf:CAP_EEEFK1E102AQ -> Capacitor_SMD:C_1206_3216Metric_Pad1.33x1.80mm_HandSolder; moved to B.Cu
- C30, C31: value 1000uF -> 1uF 400V; footprint 25V 1000uf:CAP_EEEFK1E102AQ -> Capacitor_THT:C_Rect_L24.0mm_W8.3mm_P22.50mm_MKT
- C32: value 1000uF -> 1uF 400V; footprint 25V 1000uf:CAP_EEEFK1E102AQ -> Capacitor_THT:C_Rect_L19.0mm_W9.0mm_P15.00mm_MKS4
- C33: value 1000uF -> 100n; footprint 25V 1000uf:CAP_EEEFK1E102AQ -> Capacitor_SMD:C_0805_2012Metric_Pad1.18x1.45mm_HandSolder
- C36: value 0.1uF -> 100n; footprint Capacitor_SMD:C_0201_0603Metric_Pad0.64x0.40mm_HandSolder -> Capacitor_SMD:C_0805_2012Metric_Pad1.18x1.45mm_HandSolder
- D3, D6: value 1N4007 -> US1M; moved to B.Cu
- D7, D8: value D_Snub -> MUR460
- H5: value Output - -> MountingHole_Pad; footprint MountingHole:MountingHole_6.4mm_M6_Pad -> MountingHole:MountingHole_6.4mm_M6_DIN965_Pad
- J1: footprint Connector_JST:JST_XH_S2B-XH-A_1x02_P2.50mm_Horizontal -> Connector_JST:JST_XH_B2B-XH-A_1x02_P2.50mm_Vertical
- J2: value Conn_01x04_Pin -> Conn_01x02_Male; footprint Connector_JST:JST_XH_B4B-XH-AM_1x04_P2.50mm_Vertical -> Connector_PinSocket_2.54mm:PinSocket_1x02_P2.54mm_Vertical; moved to B.Cu
- J3: value Conn_01x02_Male -> Conn_01x04_Male; footprint Connector_JST:JST_XH_S2B-XH-A_1x02_P2.50mm_Horizontal -> Connector_PinHeader_2.54mm:PinHeader_1x04_P2.54mm_Vertical
- R1, R3: value 3.3 -> 1R
- R11, R12, R13, R14, R15, R17, R18, R19, R20: value 1 -> 50mOhm 3W; moved to B.Cu
- R16: value 1 -> R_Snub 220Ohm 1W; footprint Resistor_SMD:R_2512_6332Metric_Pad1.40x3.35mm_HandSolder -> Resistor_THT:R_Box_L26.0mm_W5.0mm_P20.00mm
- R21, R23, R24, R25: value 330 -> 50mOhm 3W; footprint Resistor_SMD:R_0201_0603Metric_Pad0.64x0.40mm_HandSolder -> Resistor_SMD:R_2512_6332Metric_Pad1.40x3.35mm_HandSolder; moved to B.Cu
- R22: value 470 -> 50mOhm 3W; footprint Resistor_SMD:R_0201_0603Metric_Pad0.64x0.40mm_HandSolder -> Resistor_SMD:R_2512_6332Metric_Pad1.40x3.35mm_HandSolder; moved to B.Cu
- R5, R6: value R_Snub -> 1R; footprint Resistor_THT:R_Box_L26.0mm_W5.0mm_P20.00mm -> Resistor_SMD:R_0805_2012Metric_Pad1.20x1.40mm_HandSolder
- R7: value 22K -> R_Snub 220Ohm 1W; footprint Resistor_SMD:R_1206_3216Metric_Pad1.30x1.75mm_HandSolder -> Resistor_THT:R_Box_L26.0mm_W5.0mm_P20.00mm
- U1, U2: value LM7809_TO220 -> 78m09; footprint Package_TO_SOT_THT:TO-220-3_Vertical -> Package_TO_SOT_SMD:TO-252-2
- U10, U11: value 6N137 -> ADUM4195-1BRIZ; footprint Package_DIP:DIP-8_W7.62mm -> ADUM-4195:RI-8-1_ADI
- U3: value LM7809_TO220 -> KA78M05_TO252; footprint Package_TO_SOT_THT:TO-220-3_Vertical -> Package_TO_SOT_SMD:TO-252-2
- U4: value AMS1117-5.0 -> B0505S-1WR3; footprint Package_TO_SOT_SMD:SOT-223-3_TabPin2 -> B0505-1WR3:B0505S_MNS
- U5: value AMS1117-5.0 -> 78m09; footprint Package_TO_SOT_SMD:SOT-223-3_TabPin2 -> Package_TO_SOT_SMD:TO-252-2
- U6: value AMS1117-5.0 -> LM324; footprint Package_TO_SOT_SMD:SOT-223-3_TabPin2 -> Package_SO:SOIC-14_3.9x8.7mm_P1.27mm; moved to B.Cu
- U7: value FF150R12RT4 -> AMS1117-5.0; footprint FF300:FF300R12KS4 -> Package_TO_SOT_SMD:SOT-223-3_TabPin2
- U9: value ChinaBluePill -> ADUM4195-1BRIZ; footprint BLue Pill:ChinaBluePill -> ADUM-4195:RI-8-1_ADI
- moved C36 189.6 mm to (210.4, 194.0)
- moved R25 176.1 mm to (211.0, 188.0), turned to 180 degrees
- moved R24 174.0 mm to (211.0, 184.0), turned to 180 degrees
- moved R23 171.9 mm to (211.0, 180.0), turned to 180 degrees
- moved R22 169.9 mm to (211.0, 176.0), turned to 180 degrees
- moved R21 167.8 mm to (211.0, 172.0), turned to 180 degrees
- moved U7 163.9 mm to (116.6, 184.2), turned to 90 degrees
- moved C3 162.8 mm to (94.2, 185.5), turned to 90 degrees
- moved R11 160.7 mm to (143.2, 177.0), turned to -90 degrees
- moved C33 158.1 mm to (211.0, 196.2)
- moved C4 157.4 mm to (114.6, 192.8)
- moved R12 156.5 mm to (147.2, 177.0), turned to -90 degrees
- moved R13 152.4 mm to (151.2, 177.0), turned to -90 degrees
- moved R14 148.5 mm to (155.2, 177.0), turned to -90 degrees
- moved R15 144.7 mm to (159.2, 177.0), turned to -90 degrees
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Connections:
- C11 pad 1: Net-(U4-VO) -> Net-(U3-VO)
- C12 pad 1: Net-(U5-VO) -> VDrive1
- C13 pad 1: Net-(U6-VO) -> Net-(C13-Pad1)
- C13 pad 2: GND2 -> Net-(C13-Pad2)
- C16 pad 1: GND1 -> SensePWR
- C16 pad 2: VDrive1Neg -> DCLink-
- C17 pad 1: GND2 -> A1
- C17 pad 2: VDrive2Neg -> DCLink-
- C18 pad 1: GND1 -> DIG+
- C18 pad 2: VDrive1Neg -> DIG-
- C20 pad 2: VDrive1Neg -> GND1
- C22 pad 1: GND2 -> DIG+
- C22 pad 2: VDrive2Neg -> DIG-
- C23 pad 2: VDrive2Neg -> GND2
- C24 pad 1: Net-(D7-K) -> VDrive2
- C24 pad 2: Net-(D8-A) -> GND2
- C25 pad 1: Net-(D8-K) -> Net-(PS1-CTRL)
- C25 pad 2: DIG- -> VAux-
- C26 pad 1: +BATT -> DCLink-
- C26 pad 2: DIG- -> -BATT
- C27 pad 2: DIG- -> Net-(D7-A)
- C28 pad 1: +BATT -> Net-(D8-K)
- C28 pad 2: DIG- -> -BATT
- C29 pad 1: +BATT -> -BATT
- C29 pad 2: DIG- -> /OUT+
- C3 pad 1: Net-(PS1-CTRL) -> Net-(PS3-CTRL)
- C30 pad 1: VDrive1 -> -BATT
- C30 pad 2: GND1 -> +BATT
- C31 pad 1: GND1 -> -BATT
- C31 pad 2: VDrive1Neg -> +BATT
- C32 pad 1: VDrive2 -> -BATT
- C32 pad 2: GND2 -> /OUT+
- C33 pad 1: GND2 -> /OUTSHUNT-
- C33 pad 2: VDrive2Neg -> /OUTSHUNT+
- C36 pad 1: DIG5V -> Net-(C36-Pad1)
- C36 pad 2: DIG- -> Net-(C36-Pad2)
- C4 pad 1: Net-(PS2-CTRL) -> SensePWR
- C4 pad 2: VAux- -> DCLink-
- C5 pad 1: Net-(PS1-CTRL) -> /INSHUNT-
- C5 pad 2: VAux- -> /INSHUNT+
- C8 pad 1: Net-(U3-VO) -> VAux+
- D2 pad 2: VDrive1Neg -> GND1
- D5 pad 2: VDrive2Neg -> GND2
- D7 pad 2: +BATT -> Net-(D7-A)
- D8 pad 2: Net-(D8-A) -> Net-(D7-K)
- H5 pad 1: Net-(H5-Pad1) -> DCLink-
- IC1 pad 1: VDrive1Neg -> GND1
- IC1 pad 4: unconnected-(IC1-NC-Pad4) -> Net-(IC1-OUT-)
- IC1 pad 7: unconnected-(IC1-CLAMP-Pad7) -> Net-(IC1-CLAMP)
- IC1 pad 8: VDrive1Neg -> GND1
- IC5 pad 1: VDrive2Neg -> GND2
- IC5 pad 4: unconnected-(IC5-NC-Pad4) -> Net-(IC5-OUT-)
- IC5 pad 7: unconnected-(IC5-CLAMP-Pad7) -> Net-(IC5-CLAMP)
- IC5 pad 8: VDrive2Neg -> GND2
- J2 pad 1: Net-(J2-Pin_1) -> VAux-
- J2 pad 2: Net-(J2-Pin_2) -> VAux+
- J3 pad 1: VAux+ -> GNDCOMM
- J3 pad 2: VAux- -> RXCOMM
- Q1 pad E1: Net-(Q1-PadE1) -> GND2
- Q1 pad E2: Net-(Q1-PadE2) -> GND1
- Q1 pad E3: Net-(Q1-PadE1) -> GND2
- Q1 pad E4: Net-(Q1-PadE2) -> GND1
- Q1 pad EU1: Net-(Q1-PadEU1) -> -BATT
- Q1 pad EU2: Net-(Q1-PadEU1) -> -BATT
- Q1 pad EU3: Net-(Q1-PadEU1) -> -BATT
- Q1 pad EV1: Net-(Q1-PadEU1) -> -BATT
- Q1 pad EV2: Net-(Q1-PadEU1) -> -BATT
- Q1 pad EV3: Net-(Q1-PadEU1) -> -BATT
- Q1 pad G1: Net-(Q1-PadG1) -> Net-(IC5-CLAMP)
- Q1 pad G2: Net-(Q1-PadG2) -> Net-(IC1-CLAMP)
- Q1 pad G3: Net-(Q1-PadG1) -> Net-(IC5-CLAMP)
- Q1 pad G4: Net-(Q1-PadG2) -> Net-(IC1-CLAMP)
- Q1 pad P1: Net-(Q1-PadP1) -> +BATT
- Q1 pad P2: Net-(Q1-PadP1) -> +BATT
- Q1 pad P3: Net-(Q1-PadP1) -> +BATT
- Q1 pad T1: Net-(Q1-PadT1) -> T-
- Q1 pad T2: Net-(Q1-PadT1) -> SensePWR5V
- Q1 pad U1: Net-(Q1-PadU1) -> Net-(D7-K)
- Q1 pad U2: Net-(Q1-PadU1) -> Net-(D7-K)
- Q1 pad U3: Net-(Q1-PadU1) -> Net-(D7-K)
- Q1 pad V1: Net-(Q1-PadU1) -> Net-(D7-K)
- Q1 pad V2: Net-(Q1-PadU1) -> Net-(D7-K)
- Q1 pad V3: Net-(Q1-PadU1) -> Net-(D7-K)
- R1 pad 2: unconnected-(R1-Pad2) -> Net-(IC1-CLAMP)
- R11 pad 1: DIG- -> -BATT
- R11 pad 2: Net-(H5-Pad1) -> DCLink-
- R12 pad 1: DIG- -> -BATT
- R12 pad 2: Net-(H5-Pad1) -> DCLink-
- R13 pad 1: DIG- -> -BATT
- R13 pad 2: Net-(H5-Pad1) -> DCLink-
- R14 pad 1: DIG- -> -BATT
- R14 pad 2: Net-(H5-Pad1) -> DCLink-
- R15 pad 1: DIG- -> -BATT
- R15 pad 2: Net-(H5-Pad1) -> DCLink-
- R16 pad 1: DIG- -> -BATT
- R16 pad 2: Net-(H5-Pad1) -> Net-(D7-A)
- R17 pad 1: DIG- -> /OUT-
- R17 pad 2: Net-(H5-Pad1) -> -BATT
- R18 pad 1: DIG- -> /OUT-
- R18 pad 2: Net-(H5-Pad1) -> -BATT
- R19 pad 1: DIG- -> /OUT-
- R19 pad 2: Net-(H5-Pad1) -> -BATT
- R20 pad 1: DIG- -> /OUT-
- R20 pad 2: Net-(H5-Pad1) -> -BATT
- R21 pad 1: Net-(U10-VO) -> /OUT-
- R21 pad 2: DIG5V -> -BATT
- R22 pad 1: DIG- -> /OUT-
- R22 pad 2: Net-(U10-VO) -> -BATT
- R23 pad 1: Net-(R23-Pad1) -> /OUT-
- R23 pad 2: Net-(U11-A) -> -BATT
- R24 pad 1: Net-(J2-Pin_2) -> /OUT-
- R24 pad 2: Net-(J2-Pin_3) -> -BATT
- R25 pad 1: Net-(U10-A) -> /OUT-
- R25 pad 2: Net-(J2-Pin_4) -> -BATT
- R3 pad 2: unconnected-(R3-Pad2) -> Net-(IC5-CLAMP)
- R5 pad 1: Net-(D7-K) -> Net-(IC1-OUT-)
- R5 pad 2: +BATT -> Net-(IC1-CLAMP)
- R6 pad 1: Net-(D8-K) -> Net-(IC5-OUT-)
- R6 pad 2: Net-(D8-A) -> Net-(IC5-CLAMP)
- R7 pad 1: +BATT -> Net-(D8-K)
- R7 pad 2: DIG- -> +BATT
- U1 pad 3: Net-(PS1-CTRL) -> Net-(PS2-CTRL)
- U10 pad 1: unconnected-(U10-NC-Pad1) -> SensePWR5V
- U10 pad 2: Net-(U10-A) -> A1
- U10 pad 3: Net-(J2-Pin_1) -> DCLink-
- U10 pad 4: (no net) -> DCLink-
- U10 pad 6: Net-(U10-VO) -> DIG-
- U10 pad 7: DIG5V -> Net-(U10-VOUT)
- U11 pad 1: unconnected-(U11-NC-Pad1) -> SensePWR5V
- U11 pad 2: Net-(U11-A) -> A0
- U11 pad 3: DIG- -> DCLink-
- U11 pad 4: (no net) -> DCLink-
- U11 pad 5: Net-(J2-Pin_1) -> DIG-
- U11 pad 6: Net-(J2-Pin_3) -> DIG-
- U11 pad 7: Net-(J2-Pin_2) -> Net-(U11-VOUT)
- U11 pad 8: Net-(J2-Pin_2) -> DIG5V
- U2 pad 3: Net-(PS2-CTRL) -> Net-(PS1-CTRL)
- U4 pad 2: Net-(U4-VO) -> Net-(U3-VO)
- U4 pad 3: Net-(U3-VO) -> DIG-
- U5 pad 1: GND1 -> VAux+
- U5 pad 2: Net-(U5-VO) -> VAux-
- U5 pad 3: VDrive1 -> Net-(PS3-CTRL)
- U6 pad 1: GND2 -> Net-(R39-Pad1)
- U6 pad 2: Net-(U6-VO) -> Net-(U6A--)
- U6 pad 3: VDrive2 -> Net-(U6A-+)
- U7 pad 1: Net-(D8-A) -> DCLink-
- U7 pad 2: DIG- -> SensePWR5V
- U7 pad 3: +BATT -> SensePWR
Routing:
- net DIG-: track 0.00 -> 130.2 mm, vias 0 -> 33
- net DIG5V: track 0.00 -> 103.1 mm, vias 0 -> 12
- net Net-(Q1-PadEU1): track 92.0 -> 0.00 mm
- net Net-(Q1-PadU1): track 89.6 -> 0.00 mm
- net VAux-: track 0.00 -> 89.4 mm, vias 0 -> 7
- net /OUTSHUNT+: track 0.00 -> 86.6 mm, vias 0 -> 1
- net DIG+: track 0.00 -> 85.3 mm, vias 0 -> 11
- net /OUTSHUNT-: track 0.00 -> 82.3 mm, vias 0 -> 1
- net +BATT: track 0.00 -> 77.3 mm
- net SensePWR5V: track 0.00 -> 76.8 mm, vias 0 -> 4
- net RXD: track 0.00 -> 73.9 mm, vias 0 -> 3
- net TXD: track 0.00 -> 69.2 mm, vias 0 -> 3
- net INHS: track 0.00 -> 65.4 mm, vias 0 -> 2
- net DCLink-: track 0.00 -> 61.6 mm, vias 0 -> 7
- net GND2: track 0.00 -> 49.6 mm, vias 0 -> 5
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- added copper zone on F.Cu, net +BATT
- added copper zone on B.Cu, net -BATT
- added copper zone on F.Cu, net -BATT
- added copper zone on F.Cu, net /OUT+
- added copper zone on B.Cu, net /OUT-
- added copper zone on F.Cu, net 5VCOMM
- added copper zone on B.Cu, net DCLink-
- added copper zone on F.Cu, net DIG+
- added copper zone on B.Cu, net DIG-
- added copper zone on F.Cu, net DIG5V
- added copper zone on B.Cu, net GND1
- added copper zone on F.Cu, net GND1
- added copper zone on B.Cu, net GND2
- added copper zone on F.Cu, net GND2
- added copper zone on B.Cu, net GNDCOMM
- added copper zone on B.Cu, net Net-(D7-K)
- added copper zone on F.Cu, net Net-(D7-K)
- added copper zone on F.Cu, net SensePWR5V
- added copper zone on B.Cu, net VAux+
- added copper zone on F.Cu, net VAux-
Other:
- board outline added: 129.3 x 105.5 mm
- board text added: "3.3V"
- board text added: "5V"
- board text added: "AUX+"
- board text added: "AUX-"
- board text added: "CLK"
- board text added: "DC Link+"
- board text added: "DC Link-"
- board text added: "DIO"
- board text added: "GND"
- board text added: "OUT+"
- board text added: "OUT-"
- board text added: "RX"
- board text added: "RXD"
- board text added: "SWCLK"
- board text added: "SWDIO"
- board text added: "TX"
- board text added: "TXD"

Commit message: Final touches to LU
Parts:
- added G***: LOGO, Designed By Saksham:Designed by Saksham, F.Cu at (136.6, 96.6)
- added G***: LOGO, Designed By Saksham:vegapod_logo, F.Cu at (77.6, 36.2)
- moved D6 109.7 mm to (55.0, 26.4)
- moved R3 109.7 mm to (53.5, 35.5)
- moved R6 109.7 mm to (53.5, 37.9)
- moved C10 109.7 mm to (46.5, 28.7)
- moved C11 109.7 mm to (20.2, 47.3)
- moved C14 109.7 mm to (30.4, 40.5)
- moved C15 109.7 mm to (31.7, 33.3)
- moved C16 109.7 mm to (49.1, 109.6)
- moved C18 109.7 mm to (39.7, 36.3)
- moved C19 109.7 mm to (47.1, 55.1)
- moved C20 109.7 mm to (52.9, 61.3)
- moved C22 109.7 mm to (39.7, 56.2)
- moved C27 109.7 mm to (98.9, 18.2)
- moved C28 109.7 mm to (98.9, 71.2)
- moved C29 109.7 mm to (137.2, 32.3)
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Routing:
- net /OUTSHUNT+: track 86.6 -> 88.6 mm
Other:
- board text added: "*"
- board text added: "330uH 5.2A"
- board text added: "78M05"
- board text added: "78M09"
- board text added: "URB2415S-10WR3"
