File: Vegapod 24/Kicad Projects/7.0/BMS_Master/BMS_Master.kicad_pcb (KiCad board)
At the start: 2 copper layers, 92.6 x 87.9 mm, 87 parts, among them IC1 B0505S-2W, J1 LV Battery, J2 ST-Link, J3 Conn_01x06_Pin, K1 ECK200BHAAEA, K2 ECK200BHAAEA, Q1 SI2318CDS (SI2318), Q2 SI2318CDS (SI2318), U1 KA78M12_TO252, U11 LM324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

Commit message: BMS Master completed
Parts:
- added C33: 100n, Capacitor_SMD:C_0805_2012Metric_Pad1.18x1.45mm_HandSolder, B.Cu at (225.3, 60.1)
- added C34: 10uF, Capacitor_SMD:C_1206_3216Metric_Pad1.33x1.80mm_HandSolder, F.Cu at (246.7, 62.9)
- added C35: 10uF, Capacitor_SMD:C_1206_3216Metric_Pad1.33x1.80mm_HandSolder, B.Cu at (246.7, 60.9)
- added G***: LOGO, Logo:vegapod_logo, F.Cu at (235.3, 94.2)
- added G***: LOGO, Logo:Designed by Saksham, F.Cu at (276.2, 116.0)
- added J4: Batt Comm, Connector_PinSocket_2.00mm:PinSocket_1x05_P2.00mm_Vertical, F.Cu at (243.3, 71.6)
- added R32: 470, Resistor_SMD:R_0805_2012Metric_Pad1.20x1.40mm_HandSolder, B.Cu at (239.7, 61.2)
- added R33: 470, Resistor_SMD:R_0805_2012Metric_Pad1.20x1.40mm_HandSolder, F.Cu at (225.2, 64.0)
- added R34: 470, Resistor_SMD:R_0805_2012Metric_Pad1.20x1.40mm_HandSolder, B.Cu at (225.3, 64.1)
- added R35: 470, Resistor_SMD:R_0805_2012Metric_Pad1.20x1.40mm_HandSolder, B.Cu at (239.8, 65.6)
- added R36: 470, Resistor_SMD:R_0805_2012Metric_Pad1.20x1.40mm_HandSolder, F.Cu at (239.8, 74.1)
- added R37: 470, Resistor_SMD:R_0805_2012Metric_Pad1.20x1.40mm_HandSolder, B.Cu at (214.7, 73.6)
- added U10: 6N137, Package_SO:SSO-8_6.7x9.8mm_P2.54mm_Clearance8mm, F.Cu at (232.6, 64.0)
- added U14: 6N137, Package_SO:SSO-8_6.7x9.8mm_P2.54mm_Clearance8mm, B.Cu at (232.6, 64.0)
- added U15: B0505S-1WR3, B0505-1WR3:B0505S_MNS, F.Cu at (244.2, 67.8)
- added U16: EL814, Package_DIP:SMDIP-4_W9.53mm_Clearance8mm, B.Cu at (228.6, 72.2)
- moved C26 0.50 mm to (207.3, 72.3)
Connections:
- U13 pad 42: unconnected-(U13-PA8-Pad42) -> PA8
Routing:
- net +5VD: track 20.1 -> 92.1 mm, vias 5 -> 8
- net RX: track 0.00 -> 38.8 mm, vias 0 -> 3
- net TX: track 0.00 -> 36.9 mm, vias 0 -> 2
- net LV-: track 81.8 -> 118.4 mm, vias 28 -> 31
- net Net-(J4-Pin_2): track 0.00 -> 34.6 mm, vias 0 -> 1
- net GND1: track 0.00 -> 25.7 mm, vias 0 -> 3
- net Net-(J4-Pin_4): track 0.00 -> 13.6 mm, vias 0 -> 2
- net PA8: track 0.00 -> 9.08 mm, vias 0 -> 1
- net Net-(R37-Pad1): track 0.00 -> 9.02 mm
- net Net-(J4-Pin_5): track 0.00 -> 6.75 mm
- net Net-(J4-Pin_3): track 0.00 -> 5.21 mm
- net VD: track 58.3 -> 53.5 mm, vias 2 -> 3
- net Net-(U14-A): track 0.00 -> 3.29 mm
- net Net-(U10-A): track 0.00 -> 2.75 mm
- net LV+: track 70.1 -> 69.7 mm, vias 0 -> 2
- added copper zone on B.Cu, net GND1
- added copper zone on F.Cu, net GND1

Commit message: Flyback diode for contactor
Parts:
- added D3: US1m, Diode_SMD:D_SMA-SMB_Universal_Handsoldering, B.Cu at (240.8, 89.4)
- added D4: US1m, Diode_SMD:D_SMA-SMB_Universal_Handsoldering, F.Cu at (241.0, 105.8)
Routing:
- net LV+: track 69.7 -> 76.4 mm
- net Net-(D3-A): track 20.2 -> 22.5 mm
- net Net-(D4-A): track 30.9 -> 33.0 mm

Commit message: Add boot pin conn. (forgor💀)
Parts:
- added R38: Open Circuit, Resistor_SMD:R_0402_1005Metric, F.Cu at (199.9, 68.0)
- added R39: SHORT OUT, Resistor_SMD:R_0402_1005Metric, F.Cu at (198.9, 68.0)
- moved C27 0.22 mm to (196.1, 67.9)
Connections:
- U13 pad 61: unconnected-(U13-PB8-Pad61) -> Net-(U13-PB8)
Routing:
- net Net-(U13-PB8): track 0.00 -> 3.79 mm
- net LV-: track 118.4 -> 119.5 mm

Commit message: BMS Master changes because fucked up
Parts:
- added C36: 10uF, Capacitor_SMD:C_1206_3216Metric_Pad1.33x1.80mm_HandSolder, B.Cu at (191.4, 115.5)
- added C37: 10uF, Capacitor_SMD:C_1206_3216Metric_Pad1.33x1.80mm_HandSolder, B.Cu at (196.9, 115.5)
- added U17: B0505S-1WR3, B0505-1WR3:B0505S_MNS, F.Cu at (190.6, 117.8)
- moved C15 3.60 mm to (191.6, 111.1)
- moved C7 3.60 mm to (190.7, 107.8)
- moved U8 3.60 mm to (191.7, 105.3)
- moved D2 0.11 mm to (197.7, 108.7)
Connections:
- C11 pad 2: -BATT -> -5V
- C6 pad 2: -BATT -> -5V
- U3 pad 4: -BATT -> -5V
- U4 pad 4: -BATT -> -5V
Routing:
- net -5V: track 0.00 -> 35.1 mm, vias 0 -> 4
- net -BATT: track 62.3 -> 54.0 mm
- net +12V: track 39.8 -> 41.4 mm
- net +5V: track 10.8 -> 11.8 mm, vias 3 -> 4

Commit message: BMS Master final changes
Parts:
- added Q3: IRLZ44N, Package_TO_SOT_THT:TO-220-3_Vertical, F.Cu at (232.9, 95.9)
- added Q4: IRLZ44N, Package_TO_SOT_THT:TO-220-3_Vertical, F.Cu at (232.9, 89.9)
- moved G*** 18.2 mm to (253.3, 91.4)
Routing:
- net LV-: track 119.5 -> 135.7 mm
- net PC8: track 30.2 -> 46.1 mm
- net PC9: track 29.6 -> 43.4 mm
- net Net-(D3-A): track 22.5 -> 28.8 mm
- net Net-(D4-A): track 33.0 -> 38.3 mm
