File: Vegapod 24/Kicad Projects/7.0/BMS_LV_ADDON/BMS_LV_ADDON.kicad_pcb (KiCad board)
At the start: 2 copper layers, 85.1 x 85.1 mm, 30 parts, among them J1 Data, J2 Data, J3 DataIN, J4 DataOUT, Q1 AO3400, Q2 AO3400, Q3 AO3400, Q4 AO3400, Q5 AO3400, U1 LM393, U2 KA78M15_TO252

Commit message: BMS LV Done probably
Parts:
- added C1: Open Circuit, Capacitor_SMD:C_0603_1608Metric_Pad1.08x0.95mm_HandSolder, F.Cu at (23.4, 60.9)
- added C10: 10u, Capacitor_SMD:C_1206_3216Metric_Pad1.33x1.80mm_HandSolder, F.Cu at (55.2, 52.5)
- added C11: 100n, Capacitor_SMD:C_0805_2012Metric_Pad1.18x1.45mm_HandSolder, F.Cu at (52.2, 61.2)
- added C12: 100n, Capacitor_SMD:C_0805_2012Metric_Pad1.18x1.45mm_HandSolder, F.Cu at (45.7, 42.6)
- added C13: 10u, Capacitor_SMD:C_1206_3216Metric_Pad1.33x1.80mm_HandSolder, F.Cu at (56.4, 32.6)
- added C14: 100n, Capacitor_SMD:C_0805_2012Metric_Pad1.18x1.45mm_HandSolder, F.Cu at (50.2, 13.6)
- added C15: 100n, Capacitor_SMD:C_0805_2012Metric_Pad1.18x1.45mm_HandSolder, F.Cu at (61.4, 17.8)
- added C16: 100n, Capacitor_SMD:C_0805_2012Metric_Pad1.18x1.45mm_HandSolder, F.Cu at (45.6, 26.8)
- added C17: 100n, Capacitor_SMD:C_0805_2012Metric_Pad1.18x1.45mm_HandSolder, F.Cu at (43.8, 22.0)
- added C18: 100n, Capacitor_SMD:C_0805_2012Metric_Pad1.18x1.45mm_HandSolder, F.Cu at (56.0, 30.2)
- added C19: 10u, Capacitor_SMD:C_1206_3216Metric_Pad1.33x1.80mm_HandSolder, F.Cu at (64.4, 12.9)
- added C2: 10u, Capacitor_SMD:C_1206_3216Metric_Pad1.33x1.80mm_HandSolder, F.Cu at (2.00, 38.1)
- added C3: 10u, Capacitor_SMD:C_1206_3216Metric_Pad1.33x1.80mm_HandSolder, F.Cu at (23.1, 55.0)
- added C4: 10u, Capacitor_SMD:C_1206_3216Metric_Pad1.33x1.80mm_HandSolder, F.Cu at (11.5, 36.8)
- added C5: 10u, Capacitor_SMD:C_1206_3216Metric_Pad1.33x1.80mm_HandSolder, F.Cu at (8.60, 68.6)
- added C6: 10u, Capacitor_SMD:C_1206_3216Metric_Pad1.33x1.80mm_HandSolder, F.Cu at (7.60, 11.9)
- added C7: 10u, Capacitor_SMD:C_1206_3216Metric_Pad1.33x1.80mm_HandSolder, F.Cu at (2.20, 23.5)
- added C8: 10u, Capacitor_SMD:C_1206_3216Metric_Pad1.33x1.80mm_HandSolder, F.Cu at (11.7, 24.3)
- added C9: 10u, Capacitor_SMD:C_1206_3216Metric_Pad1.33x1.80mm_HandSolder, F.Cu at (23.0, 24.3)
- added D1: US1M, Diode_SMD:D_SMA_Handsoldering, F.Cu at (50.7, 70.1)
- added D2: US1M, Diode_SMD:D_SMA_Handsoldering, F.Cu at (50.7, 73.6)
- added D3: 5.1v Zener Diode, Diode_SMD:D_SMA_Handsoldering, F.Cu at (48.4, 39.6)
- added D4: US1M, Diode_SMD:D_SMA_Handsoldering, B.Cu at (26.6, 47.6)
- added G***: LOGO, Design:Designed by Saksham, F.Cu at (78.8, 25.2)
- added G***: LOGO, Design:vegapod_logo, F.Cu at (32.1, 32.1)
- added J10: ST-Link, Connector_PinHeader_2.54mm:PinHeader_1x04_P2.54mm_Horizontal, F.Cu at (60.7, 9.90)
- added J11: Conn_01x06_Pin, Connector_PinSocket_2.54mm:PinSocket_1x06_P2.54mm_Horizontal, F.Cu at (54.9, 10.0)
- added J5: Batt, Connector_Phoenix_MC_HighVoltage:PhoenixContact_MCV_1,5_2-G-5.08_1x02_P5.08mm_Vertical, F.Cu at (81.0, 61.0)
- added J6: Batt, Connector_Phoenix_MC_HighVoltage:PhoenixContact_MCV_1,5_2-G-5.08_1x02_P5.08mm_Vertical, F.Cu at (81.0, 49.5)
- added J7: Switch, Connector_JST:JST_XH_B2B-XH-A_1x02_P2.50mm_Vertical, F.Cu at (3.00, 47.0)
- added J8: Signal, Connector_Phoenix_MC_HighVoltage:PhoenixContact_MCV_1,5_2-G-5.08_1x02_P5.08mm_Vertical, F.Cu at (32.8, 5.74)
- added J9: OUTPUT, Connector_Phoenix_MC_HighVoltage:PhoenixContact_MCV_1,5_2-G-5.08_1x02_P5.08mm_Vertical, F.Cu at (4.00, 70.1)
- added Q6: AO3400, Package_TO_SOT_SMD:SOT-23_Handsoldering, F.Cu at (24.0, 78.4)
- added Q7: AO3400, Package_TO_SOT_SMD:SOT-23_Handsoldering, F.Cu at (27.6, 78.4)
- added Q8: AO3400, Package_TO_SOT_SMD:SOT-23_Handsoldering, F.Cu at (31.3, 78.4)
- added Q9: AO3400, Package_TO_SOT_SMD:SOT-23_Handsoldering, F.Cu at (34.9, 78.4)
- added R16: 100, Resistor_SMD:R_0603_1608Metric_Pad0.98x0.95mm_HandSolder, F.Cu at (23.0, 82.9)
- added R17: 100, Resistor_SMD:R_0603_1608Metric_Pad0.98x0.95mm_HandSolder, F.Cu at (26.6, 82.9)
- added R18: 100, Resistor_SMD:R_0603_1608Metric_Pad0.98x0.95mm_HandSolder, F.Cu at (30.3, 82.9)
- added R19: 100, Resistor_SMD:R_0603_1608Metric_Pad0.98x0.95mm_HandSolder, F.Cu at (33.9, 82.9)
- added R20: 1k, Resistor_SMD:R_0603_1608Metric_Pad0.98x0.95mm_HandSolder, F.Cu at (26.5, 61.7)
- added R21: 1k, Resistor_SMD:R_0603_1608Metric_Pad0.98x0.95mm_HandSolder, F.Cu at (35.0, 45.2)
- added R22: 100, Resistor_SMD:R_0603_1608Metric_Pad0.98x0.95mm_HandSolder, F.Cu at (51.2, 64.0)
- added R23: 100, Resistor_SMD:R_0603_1608Metric_Pad0.98x0.95mm_HandSolder, F.Cu at (53.4, 64.0)
- added R24: 100k, Resistor_SMD:R_0603_1608Metric_Pad0.98x0.95mm_HandSolder, F.Cu at (25.0, 61.7)
- added R25: 1k, Resistor_SMD:R_0603_1608Metric_Pad0.98x0.95mm_HandSolder, F.Cu at (48.8, 59.5)
- added R26: 1k, Resistor_SMD:R_0603_1608Metric_Pad0.98x0.95mm_HandSolder, F.Cu at (48.8, 58.0)
- added R27: 10k, Resistor_SMD:R_0603_1608Metric_Pad0.98x0.95mm_HandSolder, F.Cu at (47.8, 62.0)
- added R28: 10k, Resistor_SMD:R_0603_1608Metric_Pad0.98x0.95mm_HandSolder, F.Cu at (45.4, 59.4)
- added R29: 1k, Resistor_SMD:R_0603_1608Metric_Pad0.98x0.95mm_HandSolder, F.Cu at (44.6, 62.0)
- added R30: 100, Resistor_SMD:R_0603_1608Metric_Pad0.98x0.95mm_HandSolder, F.Cu at (44.6, 45.8)
- added U3: EL814, Package_DIP:SMDIP-4_W9.53mm_Clearance8mm, F.Cu at (33.7, 52.8)
- added U4: 78M05, Package_TO_SOT_SMD:TO-252-2, F.Cu at (6.97, 21.8)
- added U5: AMS1117-3.3, Package_TO_SOT_SMD:SOT-223-3_TabPin2, F.Cu at (17.4, 23.2)
- added U6: LM324, Package_SO:SOIC-14_3.9x8.7mm_P1.27mm, F.Cu at (49.3, 51.5)
- added U7: STM32G474RETx, Package_QFP:LQFP-64_10x10mm_P0.5mm, F.Cu at (52.9, 21.5)
- R1: value 15k -> 1k
- R10, R5, R6, R7, R8, R9: moved to B.Cu
- R2: value 1k -> 100
- U2: value KA78M15_TO252 -> 78M15
- moved U2 123.3 mm to (6.78, 33.9), turned to 90 degrees
- moved R3 105.7 mm to (19.9, 58.7)
- moved R4 105.5 mm to (19.8, 60.3), turned to 180 degrees
- moved U1 102.8 mm to (27.1, 56.0), turned to 90 degrees
- moved R2 99.2 mm to (28.7, 61.7), turned to 90 degrees
- moved R11 97.5 mm to (37.5, 82.9), turned to -90 degrees
- moved R1 97.4 mm to (31.3, 60.7), turned to 180 degrees
- moved Q1 94.7 mm to (38.5, 78.4), turned to 90 degrees
- moved R12 93.1 mm to (41.1, 82.9), turned to -90 degrees
- moved Q2 89.1 mm to (42.1, 78.4), turned to 90 degrees
- moved R13 88.8 mm to (44.7, 82.9), turned to -90 degrees
- moved R14 84.3 mm to (48.4, 82.9), turned to -90 degrees
- moved Q3 83.5 mm to (45.8, 78.4), turned to 90 degrees
- moved R15 79.9 mm to (52.0, 82.9), turned to -90 degrees
- moved Q4 78.0 mm to (49.4, 78.4), turned to 90 degrees
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Connections:
- net GND renamed -BATT
- net Net-(R10-Pad1) renamed SHUNT-
- net Net-(R11-Pad2) renamed Gate
- J3 pad 2: +3.3V -> unconnected-(J3-Pin_2-Pad2)
- R1 pad 1: +15V -> Net-(R1-Pad1)
- U1 pad 2: SHUNT+ -> Net-(D4-A)
- U2 pad 1: +BATT -> Net-(J7-Pin_2)
Routing:
- net SHUNT+: track 0.00 -> 162.3 mm, vias 0 -> 14
- net +BATT: track 0.00 -> 96.7 mm
- net DIN: track 0.00 -> 89.8 mm, vias 0 -> 1
- net -BATT: track 0.00 -> 78.6 mm, vias 0 -> 49
- net DOUT: track 0.00 -> 67.0 mm, vias 0 -> 1
- net Gate: track 0.00 -> 62.7 mm, vias 0 -> 2
- net Net-(D1-K): track 0.00 -> 59.0 mm
- net Net-(J8-Pin_2): track 0.00 -> 43.5 mm, vias 0 -> 1
- net Net-(J8-Pin_1): track 0.00 -> 42.5 mm, vias 0 -> 1
- net SHUNT-: track 0.00 -> 34.5 mm, vias 0 -> 1
- net +15V: track 0.00 -> 31.0 mm, vias 0 -> 1
- net A0: track 0.00 -> 25.5 mm, vias 0 -> 2
- net +3.3V: track 0.00 -> 23.7 mm
- net SCK: track 0.00 -> 19.1 mm, vias 0 -> 1
- net NSS: track 0.00 -> 18.2 mm, vias 0 -> 1
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- added copper zone on F.Cu, net +15V
- added copper zone on F.Cu, net +3.3V
- added copper zone on F.Cu, net +BATT
- added copper zone on B.Cu, net -BATT
Other:
- board text added: "*"
- board text added: "3V3"
- board text added: "BATT+"
- board text added: "BATT-"
- board text added: "CLK"
- board text added: "DIO"
- board text added: "GND"
- board text added: "MISO"
- board text added: "MOSI"
- board text added: "NC"
- board text added: "NSS"
- board text added: "OUT+"
- board text added: "OUT-"
- board text added: "SCK"
