File: Vegapod 24/Kicad Projects/7.0/BMS_LV_ADDON/BMS_LV_ADDON.kicad_sch (KiCad schematic)
At the start: 30 parts, among them J1 Data, J2 Data, J3 DataIN, J4 DataOUT, Q1 AO3400, Q2 AO3400, Q3 AO3400, Q4 AO3400, Q5 AO3400, U1 LM393, U2 KA78M15_TO252

Commit message: BMS LV Done probably
Parts:
- added C1: Open Circuit, Capacitor_SMD:C_0603_1608Metric_Pad1.08x0.95mm_HandSolder, symbol Device:C_Small
- added C10, C13, C19, C2, C3, C4, C5, C6, C7, C8, C9: 10u, Capacitor_SMD:C_1206_3216Metric_Pad1.33x1.80mm_HandSolder, symbol Device:C_Small
- added C11, C12, C14, C15, C16, C17, C18: 100n, Capacitor_SMD:C_0805_2012Metric_Pad1.18x1.45mm_HandSolder, symbol Device:C_Small
- added D1, D2, D4: US1M, Diode_SMD:D_SMA_Handsoldering, symbol Device:D_Small
- added D3: 5.1v Zener Diode, Diode_SMD:D_SMA_Handsoldering, symbol Device:D_Small
- added J2: ST-Link, Connector_PinHeader_2.54mm:PinHeader_1x04_P2.54mm_Horizontal, symbol Connector:Conn_01x04_Pin
- added J3: Conn_01x06_Pin, Connector_PinSocket_2.54mm:PinSocket_1x06_P2.54mm_Horizontal, symbol Connector:Conn_01x06_Pin
- added J5, J6: Batt, Connector_Phoenix_MC_HighVoltage:PhoenixContact_MCV_1,5_2-G-5.08_1x02_P5.08mm_Vertical, symbol Connector:Conn_01x02_Pin
- added J7: Switch, Connector_JST:JST_XH_B2B-XH-A_1x02_P2.50mm_Vertical, symbol Connector:Conn_01x02_Pin
- added J8: Signal, Connector_Phoenix_MC_HighVoltage:PhoenixContact_MCV_1,5_2-G-5.08_1x02_P5.08mm_Vertical, symbol Connector:Conn_01x02_Pin
- added J9: OUTPUT, Connector_Phoenix_MC_HighVoltage:PhoenixContact_MCV_1,5_2-G-5.08_1x02_P5.08mm_Vertical, symbol Connector:Conn_01x02_Pin
- added Q6, Q7, Q8, Q9: AO3400, Package_TO_SOT_SMD:SOT-23_Handsoldering, symbol Transistor_BJT:MMBT3904
- added R16, R17, R18, R19, R22, R23, R30: 100, Resistor_SMD:R_0603_1608Metric_Pad0.98x0.95mm_HandSolder, symbol Device:R_Small
- added R20, R21, R25, R26, R29: 1k, Resistor_SMD:R_0603_1608Metric_Pad0.98x0.95mm_HandSolder, symbol Device:R_Small
- added R24: 100k, Resistor_SMD:R_0603_1608Metric_Pad0.98x0.95mm_HandSolder, symbol Device:R_Small
- added R27, R28: 10k, Resistor_SMD:R_0603_1608Metric_Pad0.98x0.95mm_HandSolder, symbol Device:R_Small
- added U3: EL814, Package_DIP:SMDIP-4_W9.53mm_Clearance8mm, symbol Isolator:EL814
- added U4: 78M05, Package_TO_SOT_SMD:TO-252-2, symbol Regulator_Linear:KA78M05_TO252
- added U5: AMS1117-3.3, Package_TO_SOT_SMD:SOT-223-3_TabPin2, symbol Regulator_Linear:AMS1117-3.3
- added U6: LM324, Package_SO:SOIC-14_3.9x8.7mm_P1.27mm, symbol Amplifier_Operational:LM324
- added U7: STM32G474RETx, Package_QFP:LQFP-64_10x10mm_P0.5mm, symbol MCU_ST_STM32G4:STM32G474RETx
- R1: value 15k -> 1k
- R2: value 1k -> 100
- U2: value KA78M15_TO252 -> 78M15
Connections:
- net +15V: now also C10.1, C3.1, C4.1, C7.1, D4.1 (K), R24.1, U3.4, U4.1 (VI), U6.4 (V+); no longer R1.1
- net +3.3V: now also C13.1, C14.1, C15.1, C16.1, C18.1, C19.2, C6.1, C9.1, J2.4 (Pin_4), U5.2 (VO), U7.1 (VBAT), U7.16 (VDD), U7.28 (VREF+), U7.29 (VDDA), U7.32 (VDD), U7.48 (VDD), U7.64 (VDD); no longer J3.2 (Pin_2)
- net +BATT: now also C5.1, J5.2 (Pin_2), J6.2 (Pin_2), J7.1 (Pin_1), J9.2 (Pin_2); no longer U2.1 (VI)
- net DIN: now also U7.23 (PC5)
- net DOUT: now also U7.22 (PC4)
- net SHUNT+: now also D1.2 (A), D2.2 (A), Q6.2 (E), Q7.2 (E), Q8.2 (E), Q9.2 (E), R20.1, R22.2; no longer U1.2 (-)
- net Gate: now reaches R11.2, R12.2, R13.2, R14.2, R15.2, R3.2, R4.1, U1.1
- net Gate: now also R16.2, R17.2, R18.2, R19.2
- net at Q1.3 (C), Q2.3 (C), Q3.3 (C)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: now also C5.2, D1.1 (K), D2.1 (K), J9.1 (Pin_1), Q6.3 (C), Q7.3 (C), Q8.3 (C), Q9.3 (C)
- net SHUNT-: now reaches R10.1, R5.2, R6.2, R7.2, R8.1, R9.1
- net SHUNT-: now also R23.2
- net GND renamed -BATT
- net -BATT: now also C1.2, C10.2, C12.2, C13.2, C14.2, C15.2, C16.2, C17.2, C18.2, C19.1, C2.2, C3.2, C4.2, C6.2, C7.2, C8.2, C9.2, D3.2 (A), J2.1 (Pin_1), J3.6 (Pin_6), J5.1 (Pin_1), J6.1 (Pin_1), R27.1, R29.1, U4.2 (GND), U5.1 (GND), U6.11 (V-), U7.15 (VSS), U7.27 (VSSA), U7.31 (VSS), U7.47 (VSS), U7.61 (PB8), U7.63 (VSS)
- new net: R25.1, R27.2, U6.3 (+)
- new net: C11.1, R22.1, R25.2
- new net: R1.1, U3.3
- new net: R28.2, R29.2, R30.2, U6.1
- new net: C2.1, J7.2 (Pin_2), U2.1 (VI)
- new net: C11.2, R23.1, R26.2
- new net: Q9.1 (B), R19.1
- new net: R21.2, U3.1
- new net: J8.1 (Pin_1), U3.2
- new net: C1.1, D4.2 (A), R20.2, R24.2, U1.2 (-)
- new net: Q7.1 (B), R17.1
- new net: R26.1, R28.1, U6.2 (-)
- new net: C17.1, U7.7 (PG10)
- new net: J8.2 (Pin_2), R21.1
- new net: Q8.1 (B), R18.1
- new net: Q6.1 (B), R16.1
- new net +5V: C8.1, U4.3 (VO), U5.3 (VI)
- new net A0: C12.1, D3.1 (K), R30.1, U7.12 (PA0)
- new net CTRL: J3.5 (Pin_5)
- new net MISO: J3.3 (Pin_3), U7.20 (PA6)
- new net MOSI: J3.2 (Pin_2), U7.21 (PA7)
- new net NSS: J3.4 (Pin_4), U7.18 (PA4)
- new net SCK: J3.1 (Pin_1), U7.19 (PA5)
- new net SWCLK: J2.3 (Pin_3), U7.50 (PA14)
- new net SWDIO: J2.2 (Pin_2), U7.49 (PA13)
- no-connect marks 0 -> 3
